Commit message: Add 6-DOF arm integration + README

File: src/roar_simulation/urdf/arm/arm.xacro (robot description, xacro)
@@ -1,14 +1,5 @@
 <?xml version="1.0"?>
 <robot xmlns:xacro="http://www.ros.org/wiki/xacro" name="roar_arm">
-  <!--
-    This file defines the updated robotic arm and gripper as a self-contained Xacro macro.
-    - All link and joint values have been updated from the new 'roar_arm_urdf' file.
-    - Mesh paths are updated to a consistent package structure.
-    - Transmission tags are retained to define the ros_control interface.
-  -->
   <xacro:macro name="robotic_arm" params="prefix">
-    <!-- ============================================================================= -->
-    <!-- ARM LINKS AND JOINTS (Updated Values from new URDF) -->
-    <!-- ============================================================================= -->
     <link name="${prefix}base_arm">
       <inertial>
@@ -55,10 +46,9 @@
       </collision>
     </link>
-    <joint name="${prefix}joint_1" type="revolute">
+    <joint name="${prefix}joint_1" type="fixed">
       <origin xyz="0 0 0.133" rpy="0 0 0" />
       <parent link="${prefix}base_arm" />
       <child link="${prefix}link_1" />
       <axis xyz="0 0 1" />
-      <limit lower="-3.14" upper="3.14" effort="100" velocity="2" />
     </joint>
     <link name="${prefix}link_2">
@@ -84,10 +74,9 @@
       </collision>
     </link>
-    <joint name="${prefix}joint_2" type="revolute">
+    <joint name="${prefix}joint_2" type="fixed">
       <origin xyz="0.035502 0 0.1489" rpy="1.6351 -1.0672 -0.073404" />
       <parent link="${prefix}link_1" />
       <child link="${prefix}link_2" />
       <axis xyz="0.035393 0 0.99937" />
-      <limit lower="0" upper="4.71" effort="100" velocity="2" />
     </joint>
     <link name="${prefix}link_3">
@@ -113,10 +102,9 @@
       </collision>
     </link>
-    <joint name="${prefix}joint_3" type="revolute">
+    <joint name="${prefix}joint_3" type="fixed">
       <origin xyz="0 0.5275 0.1315" rpy="0 0 -1.0686" />
       <parent link="${prefix}link_2" />
       <child link="${prefix}link_3" />
       <axis xyz="0 0 -1" />
-      <limit lower="0" upper="6.28" effort="50" velocity="4" />
     </joint>
     <link name="${prefix}link_4">
@@ -142,10 +130,9 @@
       </collision>
     </link>
-    <joint name="${prefix}joint_4" type="revolute">
+    <joint name="${prefix}joint_4" type="fixed">
       <origin xyz="6.8566E-05 -0.12961 0.10761" rpy="-0.50301 1.5354 -2.073" />
       <parent link="${prefix}link_3" />
       <child link="${prefix}link_4" />
       <axis xyz="-0.031013 0 -0.99952" />
-      <limit lower="0" upper="6.28" effort="50" velocity="4" />
     </joint>
     <link name="${prefix}link_5">
@@ -171,10 +158,9 @@
       </collision>
     </link>
-    <joint name="${prefix}joint_5" type="revolute">
+    <joint name="${prefix}joint_5" type="fixed">
       <origin xyz="-0.0010256 0.083 0.10269" rpy="-1.5692 0.030978 0.050701" />
       <parent link="${prefix}link_4" />
       <child link="${prefix}link_5" />
       <axis xyz="0 0 -1" />
-      <limit lower="-3.14" upper="3.14" effort="50" velocity="4" />
     </joint>
     <link name="${prefix}link_6">
@@ -200,10 +186,9 @@
       </collision>
     </link>
-    <joint name="${prefix}joint_6" type="revolute">
-      <origin xyz="0 -0.050807 0.26285" rpy="0 0 -0.010445" />
+    <joint name="${prefix}joint_6" type="fixed">
+      <origin xyz="0 -0.050807 0.26285" rpy="0 0 1.560355" />
       <parent link="${prefix}link_5" />
       <child link="${prefix}link_6" />
       <axis xyz="0 0 -1" />
-      <limit lower="0" upper="0" effort="50" velocity="0" />
     </joint>
     <link name="${prefix}Right_ee">
@@ -229,10 +214,9 @@
       </collision>
     </link>
-    <joint name="${prefix}joint_ree" type="revolute">
+    <joint name="${prefix}joint_ree" type="fixed">
       <origin xyz="-0.030505 0.047691 -0.19085" rpy="1.5698 0 0.010445" />
       <parent link="${prefix}link_6" />
       <child link="${prefix}Right_ee" />
       <axis xyz="0 -0.0010429 1" />
-      <limit lower="0" upper="0.8" effort="15" velocity="1" />
     </joint>
     <link name="${prefix}Left_ee">
@@ -258,94 +242,10 @@
       </collision>
     </link>
-    <joint name="${prefix}joint_lee" type="revolute">
+    <joint name="${prefix}joint_lee" type="fixed">
       <origin xyz="0.029492 0.048318 -0.19085" rpy="-1.5718 0 0.010445" />
       <parent link="${prefix}link_6" />
       <child link="${prefix}Left_ee" />
       <axis xyz="0 -0.0010429 1" />
-      <limit lower="0" upper="0.8" effort="15" velocity="1" />
-    </joint>
-    <!-- ============================================================================= -->
-    <!-- TRANSMISSIONS (for ros_control) - Carried over from previous version -->
-    <!-- ============================================================================= -->
-    <transmission name="${prefix}link_1_trans">
-      <type>transmission_interface/SimpleTransmission</type>
-      <joint name="${prefix}joint_1">
-        <hardwareInterface>hardware_interface/PositionJointInterface</hardwareInterface>
-      </joint>
-      <actuator name="${prefix}link_1_motor">
-        <hardwareInterface>hardware_interface/PositionJointInterface</hardwareInterface>
-        <mechanicalReduction>1</mechanicalReduction>
-      </actuator>
-    </transmission>
-    <transmission name="${prefix}link_2_trans">
-      <type>transmission_interface/SimpleTransmission</type>
-      <joint name="${prefix}joint_2">
-        <hardwareInterface>hardware_interface/PositionJointInterface</hardwareInterface>
-      </joint>
-      <actuator name="${prefix}link_2_motor">
-        <hardwareInterface>hardware_interface/PositionJointInterface</hardwareInterface>
-        <mechanicalReduction>1</mechanicalReduction>
-      </actuator>
-    </transmission>
-    <transmission name="${prefix}link_3_trans">
-      <type>transmission_interface/SimpleTransmission</type>
-      <joint name="${prefix}joint_3">
-        <hardwareInterface>hardware_interface/PositionJointInterface</hardwareInterface>
-      </joint>
-      <actuator name="${prefix}link_3_motor">
-        <hardwareInterface>hardware_interface/PositionJointInterface</hardwareInterface>
-        <mechanicalReduction>1</mechanicalReduction>
-      </actuator>
-    </transmission>
-    <transmission name="${prefix}link_4_trans">
-      <type>transmission_interface/SimpleTransmission</type>
-      <joint name="${prefix}joint_4">
-        <hardwareInterface>hardware_interface/PositionJointInterface</hardwareInterface>
-      </joint>
-      <actuator name="${prefix}link_4_motor">
-        <hardwareInterface>hardware_interface/PositionJointInterface</hardwareInterface>
-        <mechanicalReduction>1</mechanicalReduction>
-      </actuator>
-    </transmission>
-    <transmission name="${prefix}link_5_trans">
-      <type>transmission_interface/SimpleTransmission</type>
-      <joint name="${prefix}joint_5">
-        <hardwareInterface>hardware_interface/PositionJointInterface</hardwareInterface>
-      </joint>
-      <actuator name="${prefix}link_5_motor">
-        <hardwareInterface>hardware_interface/PositionJointInterface</hardwareInterface>
-        <mechanicalReduction>1</mechanicalReduction>
-      </actuator>
-    </transmission>
-    <transmission name="${prefix}link_6_trans">
-      <type>transmission_interface/SimpleTransmission</type>
-      <joint name="${prefix}joint_6">
-        <hardwareInterface>hardware_interface/PositionJointInterface</hardwareInterface>
-      </joint>
-      <actuator name="${prefix}link_6_motor">
-        <hardwareInterface>hardware_interface/PositionJointInterface</hardwareInterface>
-        <mechanicalReduction>1</mechanicalReduction>
-      </actuator>
-    </transmission>
-    <transmission name="${prefix}Right_ee_trans">
-      <type>transmission_interface/SimpleTransmission</type>
-      <joint name="${prefix}joint_ree">
-        <hardwareInterface>hardware_interface/PositionJointInterface</hardwareInterface>
-      </joint>
-      <actuator name="${prefix}Right_ee_motor">
-        <hardwareInterface>hardware_interface/PositionJointInterface</hardwareInterface>
-        <mechanicalReduction>1</mechanicalReduction>
-      </actuator>
-    </transmission>
-    <transmission name="${prefix}Left_ee_trans">
-      <type>transmission_interface/SimpleTransmission</type>
-      <joint name="${prefix}joint_lee">
-        <hardwareInterface>hardware_interface/PositionJointInterface</hardwareInterface>
-      </joint>
-      <actuator name="${prefix}Left_ee_motor">
-        <hardwareInterface>hardware_interface/PositionJointInterface</hardwareInterface>
-        <mechanicalReduction>1</mechanicalReduction>
-      </actuator>
-    </transmission>
+    </joint>
   </xacro:macro>
 </robot>

File: src/roar_simulation/urdf/base/rover_simulation.urdf.xacro (robot description, xacro)
@@ -1,40 +1,19 @@
 <?xml version="1.0"?>
-<robot xmlns:xacro="http://www.ros.org/wiki/xacro" name="roar_simulated_rover">
-  <!--
-    ===================================================================================
-    THIS IS A ROVER-ONLY INTEGRATION FILE
-    ===================================================================================
-    Purpose: To generate a complete, stand-alone, simulatable model of the ROAR rover,
-             including its sensors and Gazebo plugins, but WITHOUT the robotic arm.
-    This file is useful for:
-      - Testing rover-specific functionalities (driving, sensors) in Gazebo.
-      - Visualizing just the rover platform in RViz.
-    It works by including our modular Xacro files and calling their macros.
-    ===================================================================================
-  -->
-  <!-- =============================================================================== -->
-  <!-- 1. INCLUDE THE REQUIRED MODULES (The "Recipe Book")                             -->
-  <!-- =============================================================================== -->
-  <!-- The physical structure of the rover (links, joints, transmissions) -->
+<robot xmlns:xacro="http://www.ros.org/wiki/name" name="roar_simulated_rover">
+  <xacro:arg name="use_gazebo" default="true" />
+  <xacro:arg name="use_hardware" default="false" />
   <xacro:include filename="$(find roar_simulation)/urdf/base/rover.xacro" />
-  <!-- The physical structure of the sensors (the camera's TF frames) -->
   <xacro:include filename="$(find roar_simulation)/urdf/modules/sensors.xacro" />
-  <!-- The simulation logic for the rover and its sensors (all Gazebo plugins) -->
+  <xacro:include filename="$(find roar_simulation)/urdf/arm/sex_dof_arm.xacro" />
   <xacro:include filename="$(find roar_simulation)/urdf/modules/rover_gazebo.xacro" />
-  <!-- =============================================================================== -->
-  <!-- 2. INSTANTIATE THE MODULES (Following the "Recipes")                            -->
-  <!-- =============================================================================== -->
-  <!-- First, build the physical rover base. -->
+  <xacro:include filename="$(find roar_simulation)/urdf/modules/arm_gazebo.xacro" />
   <xacro:rover_base />
-  <!-- Second, build and attach the physical camera structure to the rover's base_link. -->
+  <xacro:robotic_arm prefix="arm_" parent_link="arm_mount_point">
+    <origin xyz="0.0 0 0" rpy="0 0 0"/>
+  </xacro:robotic_arm>
   <xacro:depth_camera name="camera" parent_link="base_link">
-    <!-- Define the pose of the camera relative to its parent, 'base_link' -->
     <origin xyz="0 0.3 0.35" rpy="0 0 1.57079632679" />
   </xacro:depth_camera>
-  <!-- Third, attach all the Gazebo simulation plugins.
-       The plugins will find the links created by the macros above. -->
-  <!--xacro:rover_gazebo
-  controllers_yaml="$(find roar_simulation)/config/combined_controllers.yaml"/-->
-  <xacro:rover_gazebo
-  controllers_yaml="$(find roar_simulation)/config/diff_controller.yaml"/>
+  <xacro:rover_gazebo controllers_yaml="$(find roar_simulation)/config/diff_controller.yaml"/>
+  <xacro:arm_gazebo prefix="arm_" />
 </robot>

File: src/roar_simulation/urdf/modules/arm_gazebo.xacro (robot description, xacro)
@@ -2,10 +2,8 @@
 <robot xmlns:xacro="http://www.ros.org/wiki/xacro">
   <xacro:macro name="arm_gazebo" params="prefix">
-    <!-- ROS2_CONTROL HARDWARE INTERFACE FOR ARM -->
     <ros2_control name="GazeboSystemArm" type="system">
       <hardware>
         <plugin>gazebo_ros2_control/GazeboSystem</plugin>
       </hardware>
-      <!-- Arm joints - position control -->
       <joint name="${prefix}joint_1">
         <command_interface name="position">
@@ -28,6 +26,9 @@
           <param name="min">-3.14</param>
           <param name="max">3.14</param>
+          <param name="initial_value">-1.57</param>
         </command_interface>
-        <state_interface name="position"/>
+        <state_interface name="position">
+          <param name="initial_value">-1.57</param>
+        </state_interface>
         <state_interface name="velocity"/>
       </joint>
@@ -36,6 +37,9 @@
           <param name="min">-3.14</param>
           <param name="max">3.14</param>
+          <param name="initial_value">-1.57</param>
         </command_interface>
-        <state_interface name="position"/>
+        <state_interface name="position">
+          <param name="initial_value">-1.57</param>
+        </state_interface>
         <state_interface name="velocity"/>
       </joint>
@@ -44,6 +48,9 @@
           <param name="min">-3.14</param>
           <param name="max">3.14</param>
+          <param name="initial_value">0.0</param>
         </command_interface>
-        <state_interface name="position"/>
+        <state_interface name="position">
+          <param name="initial_value">0.0</param>
+        </state_interface>
         <state_interface name="velocity"/>
       </joint>
@@ -56,5 +63,4 @@
         <state_interface name="velocity"/>
       </joint>
-      <!-- End effector joints -->
       <joint name="${prefix}joint_lee">
         <command_interface name="position">
@@ -74,6 +80,5 @@
       </joint>
     </ros2_control>
-    <!-- SELF-COLLISION PROPERTIES -->
-    <gazebo reference="${prefix}base_arm">
+    <gazebo reference="${prefix}base_link">
       <selfCollide>true</selfCollide>
     </gazebo>
