Commit message: Save

File: src/roar_simulation/urdf/arm/arm.xacro (robot description, xacro)
@@ -11,14 +11,14 @@
         <origin xyz="0 0 0" rpy="0 0 0" />
         <geometry>
-          <mesh filename="package://roar_simulation/meshes/arm/base_arm.STL" />
-        </geometry>
-        <material name="">
-          <color rgba="0.79216 0.81961 0.93333 1" />
-        </material>
-      </visual>
-      <collision>
-        <origin xyz="0 0 0" rpy="0 0 0" />
-        <geometry>
-          <mesh filename="package://roar_simulation/meshes/arm/base_arm.STL" />
+          <mesh filename="package://roar_simulation/meshes/arm/base_arm_new.STL" />
+        </geometry>
+        <material name="">
+          <color rgba="0.79216 0.81961 0.93333 1" />
+        </material>
+      </visual>
+      <collision>
+        <origin xyz="0 0 0" rpy="0 0 0" />
+        <geometry>
+          <mesh filename="package://roar_simulation/meshes/arm/base_arm_new.STL" />
         </geometry>
       </collision>
@@ -33,5 +33,5 @@
         <origin xyz="0 0 0" rpy="0 0 0" />
         <geometry>
-          <mesh filename="package://roar_simulation/meshes/arm/link_1.STL" />
+          <mesh filename="package://roar_simulation/meshes/arm/link_1_new.STL" />
         </geometry>
         <material name="">
@@ -42,5 +42,5 @@
         <origin xyz="0 0 0" rpy="0 0 0" />
         <geometry>
-          <mesh filename="package://roar_simulation/meshes/arm/link_1.STL" />
+          <mesh filename="package://roar_simulation/meshes/arm/link_1_new.STL" />
         </geometry>
       </collision>
@@ -61,14 +61,14 @@
         <origin xyz="0 0 0" rpy="0 0 0" />
         <geometry>
-          <mesh filename="package://roar_simulation/meshes/arm/link_2.STL" />
-        </geometry>
-        <material name="">
-          <color rgba="0.79216 0.81961 0.93333 1" />
-        </material>
-      </visual>
-      <collision>
-        <origin xyz="0 0 0" rpy="0 0 0" />
-        <geometry>
-          <mesh filename="package://roar_simulation/meshes/arm/link_2.STL" />
+          <mesh filename="package://roar_simulation/meshes/arm/link_2_new.STL" />
+        </geometry>
+        <material name="">
+          <color rgba="0.79216 0.81961 0.93333 1" />
+        </material>
+      </visual>
+      <collision>
+        <origin xyz="0 0 0" rpy="0 0 0" />
+        <geometry>
+          <mesh filename="package://roar_simulation/meshes/arm/link_2_new.STL" />
         </geometry>
       </collision>
@@ -89,14 +89,14 @@
         <origin xyz="0 0 0" rpy="0 0 0" />
         <geometry>
-          <mesh filename="package://roar_simulation/meshes/arm/link_3.STL" />
-        </geometry>
-        <material name="">
-          <color rgba="0.79216 0.81961 0.93333 1" />
-        </material>
-      </visual>
-      <collision>
-        <origin xyz="0 0 0" rpy="0 0 0" />
-        <geometry>
-          <mesh filename="package://roar_simulation/meshes/arm/link_3.STL" />
+          <mesh filename="package://roar_simulation/meshes/arm/link_3_new.STL" />
+        </geometry>
+        <material name="">
+          <color rgba="0.79216 0.81961 0.93333 1" />
+        </material>
+      </visual>
+      <collision>
+        <origin xyz="0 0 0" rpy="0 0 0" />
+        <geometry>
+          <mesh filename="package://roar_simulation/meshes/arm/link_3_new.STL" />
         </geometry>
       </collision>
@@ -117,14 +117,14 @@
         <origin xyz="0 0 0" rpy="0 0 0" />
         <geometry>
-          <mesh filename="package://roar_simulation/meshes/arm/link_4.STL" />
-        </geometry>
-        <material name="">
-          <color rgba="0.79216 0.81961 0.93333 1" />
-        </material>
-      </visual>
-      <collision>
-        <origin xyz="0 0 0" rpy="0 0 0" />
-        <geometry>
-          <mesh filename="package://roar_simulation/meshes/arm/link_4.STL" />
+          <mesh filename="package://roar_simulation/meshes/arm/link_4_new.STL" />
+        </geometry>
+        <material name="">
+          <color rgba="0.79216 0.81961 0.93333 1" />
+        </material>
+      </visual>
+      <collision>
+        <origin xyz="0 0 0" rpy="0 0 0" />
+        <geometry>
+          <mesh filename="package://roar_simulation/meshes/arm/link_4_new.STL" />
         </geometry>
       </collision>
@@ -145,5 +145,5 @@
         <origin xyz="0 0 0" rpy="0 0 0" />
         <geometry>
-          <mesh filename="package://roar_simulation/meshes/arm/link_5.STL" />
+          <mesh filename="package://roar_simulation/meshes/arm/link_5_new.STL" />
         </geometry>
         <material name="">
@@ -154,5 +154,5 @@
         <origin xyz="0 0 0" rpy="0 0 0" />
         <geometry>
-          <mesh filename="package://roar_simulation/meshes/arm/link_5.STL" />
+          <mesh filename="package://roar_simulation/meshes/arm/link_5_new.STL" />
         </geometry>
       </collision>
@@ -173,5 +173,5 @@
         <origin xyz="0 0 0" rpy="0 0 0" />
         <geometry>
-          <mesh filename="package://roar_simulation/meshes/arm/link_6.STL" />
+          <mesh filename="package://roar_simulation/meshes/arm/link_6_new.STL" />
         </geometry>
         <material name="">
@@ -182,5 +182,5 @@
         <origin xyz="0 0 0" rpy="0 0 0" />
         <geometry>
-          <mesh filename="package://roar_simulation/meshes/arm/link_6.STL" />
+          <mesh filename="package://roar_simulation/meshes/arm/link_6_new.STL" />
         </geometry>
       </collision>

File: src/roar_simulation/urdf/base/rover.xacro (robot description, xacro)
@@ -3,10 +3,13 @@
   <xacro:include filename="$(find roar_simulation)/urdf/base/rover_control.xacro" />
   <xacro:macro name="rover_base">
-    <link name="dummy_root" />
-    <joint name="dummy_joint" type="fixed">
-      <parent link="dummy_root"/>
+    <!-- ADD THESE LINES -->
+    <link name="base_footprint"/>
+    <joint name="base_footprint_joint" type="fixed">
+      <parent link="base_footprint"/>
       <child link="base_link"/>
       <origin xyz="0 0 0" rpy="0 0 0"/>
     </joint>
+    <!-- END ADDITION -->
+    <!-- Keep everything else exactly the same below this point -->
     <link name="base_link">
       <inertial>

File: src/roar_simulation/urdf/base/rover_control.xacro (robot description, xacro)
@@ -4,5 +4,5 @@
     <ros2_control name="GazeboSimSystem" type="system">
       <hardware>
-        <plugin>gz_ros2_control/GazeboSimSystem</plugin>
+        <plugin>ign_ros2_control/IgnitionSystem</plugin>
       </hardware>
       <joint name="wheel_lhs_front_joint">

File: src/roar_simulation/urdf/base/rover_simulation.urdf.xacro (robot description, xacro)
@@ -1,4 +1,4 @@
 <?xml version="1.0"?>
-<robot xmlns:xacro="http://www.ros.org/wiki/name" name="roar_simulated_rover">
+<robot xmlns:xacro="http://www.ros.org/wiki/xacro" name="roar_simulated_rover">
   <xacro:arg name="use_gazebo" default="true" />
   <xacro:arg name="use_hardware" default="false" />
@@ -12,7 +12,12 @@
     <origin xyz="0.0 0 0" rpy="0 0 0"/>
   </xacro:robotic_arm>
-  <xacro:depth_camera name="camera" parent_link="base_link">
-    <origin xyz="0 0.3 0.35" rpy="0 0 1.57079632679" />
+  <xacro:depth_camera name="zed2i" parent_link="base_link">
+    <origin xyz="0.0 0.35 0.25" rpy="0 0 0" />
   </xacro:depth_camera>
+  <xacro:depth_camera_gazebo name="zed2i" />
+  <xacro:bno055_imu name="bno055" parent_link="base_link">
+     <origin xyz="0 0 0.1" rpy="0 0 0"/>
+  </xacro:bno055_imu>
+  <xacro:bno055_imu_gazebo name="bno055" />
   <xacro:rover_gazebo controllers_yaml="$(find roar_simulation)/config/diff_controller.yaml"/>
   <xacro:arm_gazebo prefix="arm_" />

File: src/roar_simulation/urdf/modules/rover_gazebo.xacro (robot description, xacro)
@@ -1,10 +1,158 @@
 <?xml version="1.0"?>
 <robot xmlns:xacro="http://www.ros.org/wiki/xacro">
-<xacro:macro name="rover_gazebo" params="controllers_yaml">
+  <xacro:macro name="rover_gazebo" params="controllers_yaml">
     <gazebo>
-      <plugin filename="gz_ros2_control-system" name="gz_ros2_control::GazeboSimROS2ControlPlugin">
+      <plugin filename="ign_ros2_control-system" name="ign_ros2_control::IgnitionROS2ControlPlugin">
         <parameters>${controllers_yaml}</parameters>
+      </plugin>
+      <!-- Keeping the sensors system here as a fallback, though it is also in the SDF -->
+      <plugin filename="ignition-gazebo-sensors-system" name="ignition::gazebo::systems::Sensors">
+        <render_engine>ogre2</render_engine>
       </plugin>
     </gazebo>
   </xacro:macro>
+  <xacro:macro name="depth_camera_gazebo" params="name">
+    <gazebo reference="${name}_depth_optical_frame">
+      <!-- RGB Camera -->
+      <sensor name="${name}_rgb" type="camera">
+        <update_rate>15</update_rate>
+        <topic>${name}/image_raw</topic>
+        <camera>
+          <horizontal_fov>1.91986</horizontal_fov> <!-- 110 degrees -->
+          <image><width>1280</width><height>720</height></image>
+          <clip><near>0.2</near><far>300</far></clip>
+          <noise>
+            <type>gaussian</type>
+            <mean>0.0</mean>
+            <stddev>0.007</stddev>
+          </noise>
+        </camera>
+      </sensor>
+      <!-- Depth Camera -->
+      <sensor name="${name}_depth" type="depth_camera">
+        <update_rate>15</update_rate>
+        <topic>${name}/depth</topic>
+        <camera>
+          <horizontal_fov>1.91986</horizontal_fov> <!-- 110 degrees -->
+          <image><width>1280</width><height>720</height></image>
+          <clip><near>0.2</near><far>20</far></clip>
+          <noise>
+            <type>gaussian</type>
+            <mean>0.0</mean>
+            <stddev>0.01</stddev>
+          </noise>
+        </camera>
+      </sensor>
+    </gazebo>
+  </xacro:macro>
+  <xacro:macro name="bno055_imu_gazebo" params="name">
+    <gazebo reference="${name}_link">
+      <!-- SENSOR 1: The IMU (Gyro & Accel) -->
+      <sensor name="${name}_imu_sensor" type="imu">
+        <always_on>1</always_on>
+        <update_rate>100</update_rate>
+        <visualize>true</visualize>
+        <topic>${name}/data</topic>
+        <imu>
+          <angular_velocity>
+            <x>
+              <noise type="gaussian">
+                <mean>0.0</mean>
+                <stddev>0.00173</stddev>
+                <bias_mean>0.0175</bias_mean>
+                <bias_stddev>0.001</bias_stddev>
+                <dynamic_bias_stddev>0.0005</dynamic_bias_stddev>
+                <dynamic_bias_correlation_time>400.0</dynamic_bias_correlation_time>
+              </noise>
+            </x>
+            <y>
+              <noise type="gaussian">
+                <mean>0.0</mean>
+                <stddev>0.00173</stddev>
+                <bias_mean>0.0175</bias_mean>
+                <bias_stddev>0.001</bias_stddev>
+                <dynamic_bias_stddev>0.0005</dynamic_bias_stddev>
+                <dynamic_bias_correlation_time>400.0</dynamic_bias_correlation_time>
+              </noise>
+            </y>
+            <z>
+              <noise type="gaussian">
+                <mean>0.0</mean>
+                <stddev>0.00173</stddev>
+                <bias_mean>0.0175</bias_mean>
+                <bias_stddev>0.001</bias_stddev>
+                <dynamic_bias_stddev>0.0005</dynamic_bias_stddev>
+                <dynamic_bias_correlation_time>400.0</dynamic_bias_correlation_time>
+              </noise>
+            </z>
+          </angular_velocity>
+          <linear_acceleration>
+            <x>
+              <noise type="gaussian">
+                <mean>0.0</mean>
+                <stddev>0.0104</stddev>
+                <bias_mean>0.785</bias_mean>
+                <bias_stddev>0.01</bias_stddev>
+                <dynamic_bias_stddev>0.005</dynamic_bias_stddev>
+                <dynamic_bias_correlation_time>400.0</dynamic_bias_correlation_time>
+              </noise>
+            </x>
+            <y>
+              <noise type="gaussian">
+                <mean>0.0</mean>
+                <stddev>0.0104</stddev>
+                <bias_mean>0.785</bias_mean>
+                <bias_stddev>0.01</bias_stddev>
+                <dynamic_bias_stddev>0.005</dynamic_bias_stddev>
+                <dynamic_bias_correlation_time>400.0</dynamic_bias_correlation_time>
+              </noise>
+            </y>
+            <z>
+              <noise type="gaussian">
+                <mean>0.0</mean>
+                <stddev>0.0104</stddev>
+                <bias_mean>0.785</bias_mean>
+                <bias_stddev>0.01</bias_stddev>
+                <dynamic_bias_stddev>0.005</dynamic_bias_stddev>
+                <dynamic_bias_correlation_time>400.0</dynamic_bias_correlation_time>
+              </noise>
+            </z>
+          </linear_acceleration>
+        </imu>
+      </sensor>
+      <!-- SENSOR 2: The Magnetometer -->
+      <sensor name="${name}_mag_sensor" type="magnetometer">
+        <always_on>1</always_on>
+        <update_rate>100</update_rate>
+        <visualize>true</visualize>
+        <topic>${name}/mag</topic>
+        <magnetometer>
+          <x>
+            <noise type="gaussian">
+              <mean>0.0</mean>
+              <stddev>1e-06</stddev>
+              <bias_mean>1.5e-05</bias_mean>
+              <bias_stddev>1e-06</bias_stddev>
+            </noise>
+          </x>
+          <y>
+            <noise type="gaussian">
+              <mean>0.0</mean>
+              <stddev>1e-06</stddev>
+              <bias_mean>-1.0e-05</bias_mean>
+              <bias_stddev>1e-06</bias_stddev>
+            </noise>
+          </y>
+          <z>
+            <noise type="gaussian">
+              <mean>0.0</mean>
+              <stddev>1.4e-06</stddev>
+              <bias_mean>0.5e-05</bias_mean>
+              <bias_stddev>1e-06</bias_stddev>
+            </noise>
+          </z>
+        </magnetometer>
+      </sensor>
+    </gazebo>
+  </xacro:macro>
 </robot>

File: src/roar_simulation/urdf/modules/sensors.xacro (robot description, xacro)
@@ -1,20 +1,5 @@
 <?xml version="1.0"?>
 <robot xmlns:xacro="http://www.ros.org/wiki/xacro">
-  <!--
-    This file defines the physical structure for sensors as reusable Xacro macros.
-    - It contains the links and joints needed to create the TF frames for a sensor.
-    - It does NOT contain any Gazebo plugin logic (which is in rover_gazebo.xacro).
-    - The macro is parameterized for name and mounting location for maximum flexibility.
-  -->
   <xacro:macro name="depth_camera" params="name parent_link *origin">
-    <!--
-      Macro for a depth camera's physical structure.
-      Params:
-        - name: A unique name for this camera instance (e.g., 'front_camera').
-        - parent_link: The name of the link to attach this camera to (e.g., 'base_link').
-        - *origin: An <origin> block specifying the camera's xyz and rpy offset
-                   from the parent_link.
-    -->
-    <!-- This is the main link for the camera's body. The Gazebo plugin will attach here. -->
     <link name="${name}_link">
       <inertial>
@@ -22,14 +7,25 @@
         <inertia ixx="0.0001" ixy="0.0" ixz="0.0" iyy="0.0001" iyz="0.0" izz="0.0001"/>
       </inertial>
-      <!-- This link has no <visual> or <collision> tags, making it invisible. -->
+      <visual>
+        <origin xyz="0 0 0" rpy="0 0 0"/>
+        <geometry>
+          <mesh filename="package://roar_simulation/meshes/ZED2i.stl"/>
+        </geometry>
+        <material name="camera_blue">
+          <color rgba="0.1 0.4 0.9 1.0"/>
+        </material>
+      </visual>
+      <collision>
+        <origin xyz="0 0 0" rpy="0 0 1.57079632679"/>
+        <geometry>
+          <box size="0.06 0.04 0.04"/>
+        </geometry>
+      </collision>
     </link>
-    <!-- This joint attaches the camera's body to the specified parent link. -->
     <joint name="${name}_joint" type="fixed">
       <parent link="${parent_link}" />
       <child link="${name}_link" />
-      <xacro:insert_block name="origin" /> <!-- Inserts the provided <origin> block -->
+      <xacro:insert_block name="origin" />
     </joint>
-    <!-- This is the standard optical frame for ROS cameras (Z forward, X right, Y down).
-         The Gazebo plugin will publish data relative to this frame. -->
     <link name="${name}_depth_optical_frame">
       <inertial>
@@ -38,10 +34,37 @@
       </inertial>
     </link>
-    <!-- This joint defines the standard transformation from the camera body to the optical frame. -->
     <joint name="${name}_depth_optical_joint" type="fixed">
-      <origin xyz="0 0 0" rpy="-1.57079632679 0 -1.57079632679" />
+      <origin xyz="0 0 0" rpy="0 0 1.57079632679" />
       <parent link="${name}_link" />
       <child link="${name}_depth_optical_frame" />
     </joint>
   </xacro:macro>
+  <xacro:macro name="bno055_imu" params="name parent_link *origin">
+    <link name="${name}_link">
+      <inertial>
+        <mass value="0.01"/>
+        <inertia ixx="0.0001" ixy="0.0" ixz="0.0" iyy="0.0001" iyz="0.0" izz="0.0001"/>
+      </inertial>
+      <visual>
+        <origin xyz="0 0 0" rpy="0 0 0"/>
+        <geometry>
+          <sphere radius="0.02"/>
+        </geometry>
+        <material name="imu_green">
+          <color rgba="0.1 0.9 0.1 0.5"/>
+        </material>
+      </visual>
+      <collision>
+        <origin xyz="0 0 0" rpy="0 0 0"/>
+        <geometry>
+          <sphere radius="0.02"/>
+        </geometry>
+      </collision>
+    </link>
+    <joint name="${name}_joint" type="fixed">
+      <parent link="${parent_link}" />
+      <child link="${name}_link" />
+      <xacro:insert_block name="origin" />
+    </joint>
+  </xacro:macro>
 </robot>
