Commit message: Decemenate on blender and add rover mesh files

File: src/roar_simulation/urdf/base/rover.xacro (robot description, xacro)
@@ -18,5 +18,5 @@
         <origin xyz="0 0 0" rpy="0 0 0" />
         <geometry>
-          <mesh filename="package://roar_simulation/meshes/rover/base_link.STL" />
+          <mesh filename="package://roar_simulation/meshes/rover/base_link_visual.STL" />
         </geometry>
         <material name="light_grey">
@@ -27,5 +27,5 @@
         <origin xyz="0 0 0" rpy="0 0 0" />
         <geometry>
-          <mesh filename="package://roar_simulation/meshes/rover/base_link.STL" />
+          <mesh filename="package://roar_simulation/meshes/rover/base_link_collision.STL" />
         </geometry>
       </collision>
@@ -40,5 +40,5 @@
         <origin xyz="0 0 0" rpy="0 0 0" />
         <geometry>
-          <mesh filename="package://roar_simulation/meshes/rover/rocker_rhs.STL" />
+          <mesh filename="package://roar_simulation/meshes/rover/rocker_rhs_visual.STL" />
         </geometry>
         <material name="light_blue">
@@ -49,5 +49,5 @@
         <origin xyz="0 0 0" rpy="0 0 0" />
         <geometry>
-          <mesh filename="package://roar_simulation/meshes/rover/rocker_rhs.STL" />
+          <mesh filename="package://roar_simulation/meshes/rover/rocker_rhs_collision.STL" />
         </geometry>
       </collision>
@@ -68,5 +68,5 @@
         <origin xyz="0 0 0" rpy="0 0 0" />
         <geometry>
-          <mesh filename="package://roar_simulation/meshes/rover/bogie_rhs.STL" />
+          <mesh filename="package://roar_simulation/meshes/rover/bogie_rhs_visual.STL" />
         </geometry>
         <material name="light_blue">
@@ -77,5 +77,5 @@
         <origin xyz="0 0 0" rpy="0 0 0" />
         <geometry>
-          <mesh filename="package://roar_simulation/meshes/rover/bogie_rhs.STL" />
+          <mesh filename="package://roar_simulation/meshes/rover/bogie_rhs_collision.STL" />
         </geometry>
       </collision>
@@ -105,5 +105,5 @@
         <origin xyz="0 0 0" rpy="0 0 0" />
         <geometry>
-          <mesh filename="package://roar_simulation/meshes/rover/wheel_rhs_mid.STL" />
+          <mesh filename="package://roar_simulation/meshes/rover/wheel_rhs_mid_collision.STL" />
         </geometry>
       </collision>
@@ -133,5 +133,5 @@
         <origin xyz="0 0 0" rpy="0 0 0" />
         <geometry>
-          <mesh filename="package://roar_simulation/meshes/rover/wheel_rhs_front.STL" />
+          <mesh filename="package://roar_simulation/meshes/rover/wheel_rhs_front_collision.STL" />
         </geometry>
       </collision>
@@ -161,5 +161,5 @@
         <origin xyz="0 0 0" rpy="0 0 0" />
         <geometry>
-          <mesh filename="package://roar_simulation/meshes/rover/wheel_rhs_rear.STL" />
+          <mesh filename="package://roar_simulation/meshes/rover/wheel_rhs_rear_collision.STL" />
         </geometry>
       </collision>
@@ -180,5 +180,5 @@
         <origin xyz="0 0 0" rpy="0 0 0" />
         <geometry>
-          <mesh filename="package://roar_simulation/meshes/rover/rocker_lhs.STL" />
+          <mesh filename="package://roar_simulation/meshes/rover/rocker_lhs_visual.STL" />
         </geometry>
         <material name="light_blue">
@@ -189,5 +189,5 @@
         <origin xyz="0 0 0" rpy="0 0 0" />
         <geometry>
-          <mesh filename="package://roar_simulation/meshes/rover/rocker_lhs.STL" />
+          <mesh filename="package://roar_simulation/meshes/rover/rocker_lhs_collision.STL" />
         </geometry>
       </collision>
@@ -208,5 +208,5 @@
         <origin xyz="0 0 0" rpy="0 0 0" />
         <geometry>
-          <mesh filename="package://roar_simulation/meshes/rover/bogie_lhs.STL" />
+          <mesh filename="package://roar_simulation/meshes/rover/bogie_lhs_visual.STL" />
         </geometry>
         <material name="light_blue">
@@ -217,5 +217,5 @@
         <origin xyz="0 0 0" rpy="0 0 0" />
         <geometry>
-          <mesh filename="package://roar_simulation/meshes/rover/bogie_lhs.STL" />
+          <mesh filename="package://roar_simulation/meshes/rover/bogie_lhs_collision.STL" />
         </geometry>
       </collision>
@@ -245,5 +245,5 @@
         <origin xyz="0 0 0" rpy="0 0 0" />
         <geometry>
-          <mesh filename="package://roar_simulation/meshes/rover/wheel_lhs_mid.STL" />
+          <mesh filename="package://roar_simulation/meshes/rover/wheel_lhs_mid_collision.STL" />
         </geometry>
       </collision>
@@ -273,5 +273,5 @@
         <origin xyz="0 0 0" rpy="0 0 0" />
         <geometry>
-          <mesh filename="package://roar_simulation/meshes/rover/wheel_lhs_front.STL" />
+          <mesh filename="package://roar_simulation/meshes/rover/wheel_lhs_front_collision.STL" />
         </geometry>
       </collision>
@@ -301,5 +301,5 @@
         <origin xyz="0 0 0" rpy="0 0 0" />
         <geometry>
-          <mesh filename="package://roar_simulation/meshes/rover/wheel_lhs_rear.STL" />
+          <mesh filename="package://roar_simulation/meshes/rover/wheel_lhs_rear_collision.STL" />
         </geometry>
       </collision>
