Commit message: Fix ros2_control plugin compatibility and upload rover meshes

File: src/roar_simulation/urdf/modules/rover_gazebo.xacro (robot description, xacro)
@@ -3,5 +3,5 @@
   <xacro:macro name="rover_gazebo" params="controllers_yaml">
     <gazebo>
-      <plugin filename="ign_ros2_control-system" name="ign_ros2_control::IgnitionROS2ControlPlugin">
+      <plugin filename="gz_ros2_control-system" name="gz_ros2_control::GazeboSimROS2ControlPlugin">
         <parameters>${controllers_yaml}</parameters>
       </plugin>

File: src/roar_simulation/urdf/modules/sensors.xacro (robot description, xacro)
@@ -10,5 +10,6 @@
         <origin xyz="0 0 0" rpy="0 0 0"/>
         <geometry>
-          <mesh filename="package://roar_simulation/meshes/ZED2i.stl"/>
+          <!-- ZED2i mesh is not present in this package; use a simple fallback visual -->
+          <box size="0.08 0.04 0.06"/>
         </geometry>
         <material name="camera_blue">
