Commit message: updated rover with correctly working movement (robot description wise)

File: rover/roar_rover_clean/urdf/base/rover.xacro (robot description, xacro)
@@ -1,6 +1,12 @@
 <?xml version="1.0"?>
 <robot xmlns:xacro="http://www.ros.org/wiki/xacro" name="roar_rover">
-  <xacro:include filename="$(find roar_rover_clean)/urdf/base/rover_control.xacro" />
+  <xacro:include filename="$(find roar_simulation_full)/urdf/base/rover_control.xacro" />
   <xacro:macro name="rover_base">
+    <link name="base_footprint"/>
+    <joint name="base_footprint_joint" type="fixed">
+      <parent link="base_footprint"/>
+      <child link="base_link"/>
+      <origin xyz="0 0 0" rpy="0 0 -1.57079632679"/>
+    </joint>
     <link name="base_link">
       <inertial>
@@ -12,5 +18,5 @@
         <origin xyz="0 0 0" rpy="0 0 0" />
         <geometry>
-          <mesh filename="file://$(find roar_rover_clean)/meshes/rover/base_link_visual.STL" />
+          <mesh filename="file://$(find roar_simulation_full)/meshes/rover/base_link_visual.STL" />
         </geometry>
         <material name="light_grey">
@@ -21,5 +27,5 @@
         <origin xyz="0 0 0" rpy="0 0 0" />
         <geometry>
-          <mesh filename="file://$(find roar_rover_clean)/meshes/rover/base_link_collision.STL" />
+          <mesh filename="file://$(find roar_simulation_full)/meshes/rover/base_link_collision.STL" />
         </geometry>
       </collision>
@@ -34,5 +40,5 @@
         <origin xyz="0 0 0" rpy="0 0 0" />
         <geometry>
-          <mesh filename="file://$(find roar_rover_clean)/meshes/rover/rocker_rhs_visual.STL" />
+          <mesh filename="file://$(find roar_simulation_full)/meshes/rover/rocker_rhs_visual.STL" />
         </geometry>
         <material name="light_blue">
@@ -43,5 +49,5 @@
         <origin xyz="0 0 0" rpy="0 0 0" />
         <geometry>
-          <mesh filename="file://$(find roar_rover_clean)/meshes/rover/rocker_rhs_collision.STL" />
+          <mesh filename="file://$(find roar_simulation_full)/meshes/rover/rocker_rhs_collision.STL" />
         </geometry>
       </collision>
@@ -62,5 +68,5 @@
         <origin xyz="0 0 0" rpy="0 0 0" />
         <geometry>
-          <mesh filename="file://$(find roar_rover_clean)/meshes/rover/bogie_rhs_visual.STL" />
+          <mesh filename="file://$(find roar_simulation_full)/meshes/rover/bogie_rhs_visual.STL" />
         </geometry>
         <material name="light_blue">
@@ -71,5 +77,5 @@
         <origin xyz="0 0 0" rpy="0 0 0" />
         <geometry>
-          <mesh filename="file://$(find roar_rover_clean)/meshes/rover/bogie_rhs_collision.STL" />
+          <mesh filename="file://$(find roar_simulation_full)/meshes/rover/bogie_rhs_collision.STL" />
         </geometry>
       </collision>
@@ -90,14 +96,14 @@
         <origin xyz="0 0 0" rpy="0 0 0" />
         <geometry>
-          <mesh filename="file://$(find roar_rover_clean)/meshes/rover/wheel_rhs_mid.STL" />
-        </geometry>
-        <material name="dark_grey">
-          <color rgba="0.29803 0.29803 0.29803 1" />
-        </material>
-      </visual>
-      <collision>
-        <origin xyz="0 0 0" rpy="0 0 0" />
-        <geometry>
-          <mesh filename="file://$(find roar_rover_clean)/meshes/rover/wheel_rhs_mid_collision.STL" />
+          <mesh filename="file://$(find roar_simulation_full)/meshes/rover/wheel_rhs_mid.STL" />
+        </geometry>
+        <material name="dark_grey">
+          <color rgba="0.29803 0.29803 0.29803 1" />
+        </material>
+      </visual>
+      <collision>
+        <origin xyz="0 0 0" rpy="0 0 0" />
+        <geometry>
+          <mesh filename="file://$(find roar_simulation_full)/meshes/rover/wheel_rhs_mid_collision.STL" />
         </geometry>
       </collision>
@@ -118,14 +124,14 @@
         <origin xyz="0 0 0" rpy="0 0 0" />
         <geometry>
-          <mesh filename="file://$(find roar_rover_clean)/meshes/rover/wheel_rhs_front.STL" />
-        </geometry>
-        <material name="dark_grey">
-          <color rgba="0.29803 0.29803 0.29803 1" />
-        </material>
-      </visual>
-      <collision>
-        <origin xyz="0 0 0" rpy="0 0 0" />
-        <geometry>
-          <mesh filename="file://$(find roar_rover_clean)/meshes/rover/wheel_rhs_front_collision.STL" />
+          <mesh filename="file://$(find roar_simulation_full)/meshes/rover/wheel_rhs_front.STL" />
+        </geometry>
+        <material name="dark_grey">
+          <color rgba="0.29803 0.29803 0.29803 1" />
+        </material>
+      </visual>
+      <collision>
+        <origin xyz="0 0 0" rpy="0 0 0" />
+        <geometry>
+          <mesh filename="file://$(find roar_simulation_full)/meshes/rover/wheel_rhs_front_collision.STL" />
         </geometry>
       </collision>
@@ -146,14 +152,14 @@
         <origin xyz="0 0 0" rpy="0 0 0" />
         <geometry>
-          <mesh filename="file://$(find roar_rover_clean)/meshes/rover/wheel_rhs_rear.STL" />
-        </geometry>
-        <material name="dark_grey">
-          <color rgba="0.29803 0.29803 0.29803 1" />
-        </material>
-      </visual>
-      <collision>
-        <origin xyz="0 0 0" rpy="0 0 0" />
-        <geometry>
-          <mesh filename="file://$(find roar_rover_clean)/meshes/rover/wheel_rhs_rear_collision.STL" />
+          <mesh filename="file://$(find roar_simulation_full)/meshes/rover/wheel_rhs_rear.STL" />
+        </geometry>
+        <material name="dark_grey">
+          <color rgba="0.29803 0.29803 0.29803 1" />
+        </material>
+      </visual>
+      <collision>
+        <origin xyz="0 0 0" rpy="0 0 0" />
+        <geometry>
+          <mesh filename="file://$(find roar_simulation_full)/meshes/rover/wheel_rhs_rear_collision.STL" />
         </geometry>
       </collision>
@@ -174,5 +180,5 @@
         <origin xyz="0 0 0" rpy="0 0 0" />
         <geometry>
-          <mesh filename="file://$(find roar_rover_clean)/meshes/rover/rocker_lhs_visual.STL" />
+          <mesh filename="file://$(find roar_simulation_full)/meshes/rover/rocker_lhs_visual.STL" />
         </geometry>
         <material name="light_blue">
@@ -183,5 +189,5 @@
         <origin xyz="0 0 0" rpy="0 0 0" />
         <geometry>
-          <mesh filename="file://$(find roar_rover_clean)/meshes/rover/rocker_lhs.STL" />
+          <mesh filename="file://$(find roar_simulation_full)/meshes/rover/rocker_lhs.STL" />
         </geometry>
       </collision>
@@ -202,5 +208,5 @@
         <origin xyz="0 0 0" rpy="0 0 0" />
         <geometry>
-          <mesh filename="file://$(find roar_rover_clean)/meshes/rover/bogie_lhs_visual.STL" />
+          <mesh filename="file://$(find roar_simulation_full)/meshes/rover/bogie_lhs_visual.STL" />
         </geometry>
         <material name="light_blue">
@@ -211,5 +217,5 @@
         <origin xyz="0 0 0" rpy="0 0 0" />
         <geometry>
-          <mesh filename="file://$(find roar_rover_clean)/meshes/rover/bogie_lhs_collision.STL" />
+          <mesh filename="file://$(find roar_simulation_full)/meshes/rover/bogie_lhs_collision.STL" />
         </geometry>
       </collision>
@@ -230,14 +236,14 @@
         <origin xyz="0 0 0" rpy="0 0 0" />
         <geometry>
-          <mesh filename="file://$(find roar_rover_clean)/meshes/rover/wheel_lhs_mid.STL" />
-        </geometry>
-        <material name="dark_grey">
-          <color rgba="0.29803 0.29803 0.29803 1" />
-        </material>
-      </visual>
-      <collision>
-        <origin xyz="0 0 0" rpy="0 0 0" />
-        <geometry>
-          <mesh filename="file://$(find roar_rover_clean)/meshes/rover/wheel_lhs_mid_collision.STL" />
+          <mesh filename="file://$(find roar_simulation_full)/meshes/rover/wheel_lhs_mid.STL" />
+        </geometry>
+        <material name="dark_grey">
+          <color rgba="0.29803 0.29803 0.29803 1" />
+        </material>
+      </visual>
+      <collision>
+        <origin xyz="0 0 0" rpy="0 0 0" />
+        <geometry>
+          <mesh filename="file://$(find roar_simulation_full)/meshes/rover/wheel_lhs_mid_collision.STL" />
         </geometry>
       </collision>
@@ -258,14 +264,14 @@
         <origin xyz="0 0 0" rpy="0 0 0" />
         <geometry>
-          <mesh filename="file://$(find roar_rover_clean)/meshes/rover/wheel_lhs_front.STL" />
-        </geometry>
-        <material name="dark_grey">
-          <color rgba="0.29803 0.29803 0.29803 1" />
-        </material>
-      </visual>
-      <collision>
-        <origin xyz="0 0 0" rpy="0 0 0" />
-        <geometry>
-          <mesh filename="file://$(find roar_rover_clean)/meshes/rover/wheel_lhs_front_collision.STL" />
+          <mesh filename="file://$(find roar_simulation_full)/meshes/rover/wheel_lhs_front.STL" />
+        </geometry>
+        <material name="dark_grey">
+          <color rgba="0.29803 0.29803 0.29803 1" />
+        </material>
+      </visual>
+      <collision>
+        <origin xyz="0 0 0" rpy="0 0 0" />
+        <geometry>
+          <mesh filename="file://$(find roar_simulation_full)/meshes/rover/wheel_lhs_front_collision.STL" />
         </geometry>
       </collision>
@@ -286,14 +292,14 @@
         <origin xyz="0 0 0" rpy="0 0 0" />
         <geometry>
-          <mesh filename="file://$(find roar_rover_clean)/meshes/rover/wheel_lhs_rear.STL" />
-        </geometry>
-        <material name="dark_grey">
-          <color rgba="0.29803 0.29803 0.29803 1" />
-        </material>
-      </visual>
-      <collision>
-        <origin xyz="0 0 0" rpy="0 0 0" />
-        <geometry>
-          <mesh filename="file://$(find roar_rover_clean)/meshes/rover/wheel_lhs_rear_collision.STL" />
+          <mesh filename="file://$(find roar_simulation_full)/meshes/rover/wheel_lhs_rear.STL" />
+        </geometry>
+        <material name="dark_grey">
+          <color rgba="0.29803 0.29803 0.29803 1" />
+        </material>
+      </visual>
+      <collision>
+        <origin xyz="0 0 0" rpy="0 0 0" />
+        <geometry>
+          <mesh filename="file://$(find roar_simulation_full)/meshes/rover/wheel_lhs_rear_collision.STL" />
         </geometry>
       </collision>

File: rover/roar_rover_clean/urdf/modules/rover_gazebo.xacro (robot description, xacro)
@@ -5,18 +5,4 @@
       <plugin filename="ign_ros2_control-system" name="ign_ros2_control::IgnitionROS2ControlPlugin">
         <parameters>${controllers_yaml}</parameters>
-      </plugin>
-      <plugin
-        filename="ignition-gazebo-diff-drive-system"
-        name="ignition::gazebo::systems::DiffDrive">
-        <left_joint>wheel_lhs_front_joint</left_joint>
-        <left_joint>wheel_lhs_mid_joint</left_joint>
-        <left_joint>wheel_lhs_rear_joint</left_joint>
-        <right_joint>wheel_rhs_front_joint</right_joint>
-        <right_joint>wheel_rhs_mid_joint</right_joint>
-        <right_joint>wheel_rhs_rear_joint</right_joint>
-        <wheel_separation>0.61</wheel_separation>
-        <wheel_radius>0.1</wheel_radius>
-        <odom_publish_frequency>50</odom_publish_frequency>
-        <topic>cmd_vel</topic>
       </plugin>
     </gazebo>

File: rover/roar_rover_clean/urdf/modules/rover_gazebo_clean.xacro (robot description, xacro)
@@ -5,18 +5,4 @@
       <plugin filename="ign_ros2_control-system" name="ign_ros2_control::IgnitionROS2ControlPlugin">
         <parameters>${controllers_yaml}</parameters>
-      </plugin>
-      <plugin
-        filename="ignition-gazebo-diff-drive-system"
-        name="ignition::gazebo::systems::DiffDrive">
-        <left_joint>wheel_lhs_front_joint</left_joint>
-        <left_joint>wheel_lhs_mid_joint</left_joint>
-        <left_joint>wheel_lhs_rear_joint</left_joint>
-        <right_joint>wheel_rhs_front_joint</right_joint>
-        <right_joint>wheel_rhs_mid_joint</right_joint>
-        <right_joint>wheel_rhs_rear_joint</right_joint>
-        <wheel_separation>0.61</wheel_separation>
-        <wheel_radius>0.1</wheel_radius>
-        <odom_publish_frequency>50</odom_publish_frequency>
-        <topic>cmd_vel</topic>
       </plugin>
     </gazebo>

File: rover/roar_rover_noise/urdf/base/rover.xacro (robot description, xacro)
@@ -1,6 +1,12 @@
 <?xml version="1.0"?>
 <robot xmlns:xacro="http://www.ros.org/wiki/xacro" name="roar_rover">
-  <xacro:include filename="$(find roar_rover_noise)/urdf/base/rover_control.xacro" />
+  <xacro:include filename="$(find roar_simulation_full)/urdf/base/rover_control.xacro" />
   <xacro:macro name="rover_base">
+    <link name="base_footprint"/>
+    <joint name="base_footprint_joint" type="fixed">
+      <parent link="base_footprint"/>
+      <child link="base_link"/>
+      <origin xyz="0 0 0" rpy="0 0 -1.57079632679"/>
+    </joint>
     <link name="base_link">
       <inertial>
@@ -12,5 +18,5 @@
         <origin xyz="0 0 0" rpy="0 0 0" />
         <geometry>
-          <mesh filename="file://$(find roar_rover_noise)/meshes/rover/base_link_visual.STL" />
+          <mesh filename="file://$(find roar_simulation_full)/meshes/rover/base_link_visual.STL" />
         </geometry>
         <material name="light_grey">
@@ -21,5 +27,5 @@
         <origin xyz="0 0 0" rpy="0 0 0" />
         <geometry>
-          <mesh filename="file://$(find roar_rover_noise)/meshes/rover/base_link_collision.STL" />
+          <mesh filename="file://$(find roar_simulation_full)/meshes/rover/base_link_collision.STL" />
         </geometry>
       </collision>
@@ -34,5 +40,5 @@
         <origin xyz="0 0 0" rpy="0 0 0" />
         <geometry>
-          <mesh filename="file://$(find roar_rover_noise)/meshes/rover/rocker_rhs_visual.STL" />
+          <mesh filename="file://$(find roar_simulation_full)/meshes/rover/rocker_rhs_visual.STL" />
         </geometry>
         <material name="light_blue">
@@ -43,5 +49,5 @@
         <origin xyz="0 0 0" rpy="0 0 0" />
         <geometry>
-          <mesh filename="file://$(find roar_rover_noise)/meshes/rover/rocker_rhs_collision.STL" />
+          <mesh filename="file://$(find roar_simulation_full)/meshes/rover/rocker_rhs_collision.STL" />
         </geometry>
       </collision>
@@ -62,5 +68,5 @@
         <origin xyz="0 0 0" rpy="0 0 0" />
         <geometry>
-          <mesh filename="file://$(find roar_rover_noise)/meshes/rover/bogie_rhs_visual.STL" />
+          <mesh filename="file://$(find roar_simulation_full)/meshes/rover/bogie_rhs_visual.STL" />
         </geometry>
         <material name="light_blue">
@@ -71,5 +77,5 @@
         <origin xyz="0 0 0" rpy="0 0 0" />
         <geometry>
-          <mesh filename="file://$(find roar_rover_noise)/meshes/rover/bogie_rhs_collision.STL" />
+          <mesh filename="file://$(find roar_simulation_full)/meshes/rover/bogie_rhs_collision.STL" />
         </geometry>
       </collision>
@@ -90,14 +96,14 @@
         <origin xyz="0 0 0" rpy="0 0 0" />
         <geometry>
-          <mesh filename="file://$(find roar_rover_noise)/meshes/rover/wheel_rhs_mid.STL" />
-        </geometry>
-        <material name="dark_grey">
-          <color rgba="0.29803 0.29803 0.29803 1" />
-        </material>
-      </visual>
-      <collision>
-        <origin xyz="0 0 0" rpy="0 0 0" />
-        <geometry>
-          <mesh filename="file://$(find roar_rover_noise)/meshes/rover/wheel_rhs_mid_collision.STL" />
+          <mesh filename="file://$(find roar_simulation_full)/meshes/rover/wheel_rhs_mid.STL" />
+        </geometry>
+        <material name="dark_grey">
+          <color rgba="0.29803 0.29803 0.29803 1" />
+        </material>
+      </visual>
+      <collision>
+        <origin xyz="0 0 0" rpy="0 0 0" />
+        <geometry>
+          <mesh filename="file://$(find roar_simulation_full)/meshes/rover/wheel_rhs_mid_collision.STL" />
         </geometry>
       </collision>
@@ -118,14 +124,14 @@
         <origin xyz="0 0 0" rpy="0 0 0" />
         <geometry>
-          <mesh filename="file://$(find roar_rover_noise)/meshes/rover/wheel_rhs_front.STL" />
-        </geometry>
-        <material name="dark_grey">
-          <color rgba="0.29803 0.29803 0.29803 1" />
-        </material>
-      </visual>
-      <collision>
-        <origin xyz="0 0 0" rpy="0 0 0" />
-        <geometry>
-          <mesh filename="file://$(find roar_rover_noise)/meshes/rover/wheel_rhs_front_collision.STL" />
+          <mesh filename="file://$(find roar_simulation_full)/meshes/rover/wheel_rhs_front.STL" />
+        </geometry>
+        <material name="dark_grey">
+          <color rgba="0.29803 0.29803 0.29803 1" />
+        </material>
+      </visual>
+      <collision>
+        <origin xyz="0 0 0" rpy="0 0 0" />
+        <geometry>
+          <mesh filename="file://$(find roar_simulation_full)/meshes/rover/wheel_rhs_front_collision.STL" />
         </geometry>
       </collision>
@@ -146,14 +152,14 @@
         <origin xyz="0 0 0" rpy="0 0 0" />
         <geometry>
-          <mesh filename="file://$(find roar_rover_noise)/meshes/rover/wheel_rhs_rear.STL" />
-        </geometry>
-        <material name="dark_grey">
-          <color rgba="0.29803 0.29803 0.29803 1" />
-        </material>
-      </visual>
-      <collision>
-        <origin xyz="0 0 0" rpy="0 0 0" />
-        <geometry>
-          <mesh filename="file://$(find roar_rover_noise)/meshes/rover/wheel_rhs_rear_collision.STL" />
+          <mesh filename="file://$(find roar_simulation_full)/meshes/rover/wheel_rhs_rear.STL" />
+        </geometry>
+        <material name="dark_grey">
+          <color rgba="0.29803 0.29803 0.29803 1" />
+        </material>
+      </visual>
+      <collision>
+        <origin xyz="0 0 0" rpy="0 0 0" />
+        <geometry>
+          <mesh filename="file://$(find roar_simulation_full)/meshes/rover/wheel_rhs_rear_collision.STL" />
         </geometry>
       </collision>
@@ -174,5 +180,5 @@
         <origin xyz="0 0 0" rpy="0 0 0" />
         <geometry>
-          <mesh filename="file://$(find roar_rover_noise)/meshes/rover/rocker_lhs_visual.STL" />
+          <mesh filename="file://$(find roar_simulation_full)/meshes/rover/rocker_lhs_visual.STL" />
         </geometry>
         <material name="light_blue">
@@ -183,5 +189,5 @@
         <origin xyz="0 0 0" rpy="0 0 0" />
         <geometry>
-          <mesh filename="file://$(find roar_rover_noise)/meshes/rover/rocker_lhs.STL" />
+          <mesh filename="file://$(find roar_simulation_full)/meshes/rover/rocker_lhs.STL" />
         </geometry>
       </collision>
@@ -202,5 +208,5 @@
         <origin xyz="0 0 0" rpy="0 0 0" />
         <geometry>
-          <mesh filename="file://$(find roar_rover_noise)/meshes/rover/bogie_lhs_visual.STL" />
+          <mesh filename="file://$(find roar_simulation_full)/meshes/rover/bogie_lhs_visual.STL" />
         </geometry>
         <material name="light_blue">
@@ -211,5 +217,5 @@
         <origin xyz="0 0 0" rpy="0 0 0" />
         <geometry>
-          <mesh filename="file://$(find roar_rover_noise)/meshes/rover/bogie_lhs_collision.STL" />
+          <mesh filename="file://$(find roar_simulation_full)/meshes/rover/bogie_lhs_collision.STL" />
         </geometry>
       </collision>
@@ -230,14 +236,14 @@
         <origin xyz="0 0 0" rpy="0 0 0" />
         <geometry>
-          <mesh filename="file://$(find roar_rover_noise)/meshes/rover/wheel_lhs_mid.STL" />
-        </geometry>
-        <material name="dark_grey">
-          <color rgba="0.29803 0.29803 0.29803 1" />
-        </material>
-      </visual>
-      <collision>
-        <origin xyz="0 0 0" rpy="0 0 0" />
-        <geometry>
-          <mesh filename="file://$(find roar_rover_noise)/meshes/rover/wheel_lhs_mid_collision.STL" />
+          <mesh filename="file://$(find roar_simulation_full)/meshes/rover/wheel_lhs_mid.STL" />
+        </geometry>
+        <material name="dark_grey">
+          <color rgba="0.29803 0.29803 0.29803 1" />
+        </material>
+      </visual>
+      <collision>
+        <origin xyz="0 0 0" rpy="0 0 0" />
+        <geometry>
+          <mesh filename="file://$(find roar_simulation_full)/meshes/rover/wheel_lhs_mid_collision.STL" />
         </geometry>
       </collision>
@@ -258,14 +264,14 @@
         <origin xyz="0 0 0" rpy="0 0 0" />
         <geometry>
-          <mesh filename="file://$(find roar_rover_noise)/meshes/rover/wheel_lhs_front.STL" />
-        </geometry>
-        <material name="dark_grey">
-          <color rgba="0.29803 0.29803 0.29803 1" />
-        </material>
-      </visual>
-      <collision>
-        <origin xyz="0 0 0" rpy="0 0 0" />
-        <geometry>
-          <mesh filename="file://$(find roar_rover_noise)/meshes/rover/wheel_lhs_front_collision.STL" />
+          <mesh filename="file://$(find roar_simulation_full)/meshes/rover/wheel_lhs_front.STL" />
+        </geometry>
+        <material name="dark_grey">
+          <color rgba="0.29803 0.29803 0.29803 1" />
+        </material>
+      </visual>
+      <collision>
+        <origin xyz="0 0 0" rpy="0 0 0" />
+        <geometry>
+          <mesh filename="file://$(find roar_simulation_full)/meshes/rover/wheel_lhs_front_collision.STL" />
         </geometry>
       </collision>
@@ -286,14 +292,14 @@
         <origin xyz="0 0 0" rpy="0 0 0" />
         <geometry>
-          <mesh filename="file://$(find roar_rover_noise)/meshes/rover/wheel_lhs_rear.STL" />
-        </geometry>
-        <material name="dark_grey">
-          <color rgba="0.29803 0.29803 0.29803 1" />
-        </material>
-      </visual>
-      <collision>
-        <origin xyz="0 0 0" rpy="0 0 0" />
-        <geometry>
-          <mesh filename="file://$(find roar_rover_noise)/meshes/rover/wheel_lhs_rear_collision.STL" />
+          <mesh filename="file://$(find roar_simulation_full)/meshes/rover/wheel_lhs_rear.STL" />
+        </geometry>
+        <material name="dark_grey">
+          <color rgba="0.29803 0.29803 0.29803 1" />
+        </material>
+      </visual>
+      <collision>
+        <origin xyz="0 0 0" rpy="0 0 0" />
+        <geometry>
+          <mesh filename="file://$(find roar_simulation_full)/meshes/rover/wheel_lhs_rear_collision.STL" />
         </geometry>
       </collision>

File: rover/roar_simulation_full/urdf/base/rover.xacro (robot description, xacro)
@@ -3,4 +3,10 @@
   <xacro:include filename="$(find roar_simulation_full)/urdf/base/rover_control.xacro" />
   <xacro:macro name="rover_base">
+    <link name="base_footprint"/>
+    <joint name="base_footprint_joint" type="fixed">
+      <parent link="base_footprint"/>
+      <child link="base_link"/>
+      <origin xyz="0 0 0" rpy="0 0 -1.57079632679"/>
+    </joint>
     <link name="base_link">
       <inertial>
