Commit message: Update panel ros2control configurations and xacro scope placement

File: panel/final_panel.urdf (robot description, URDF)
Before this commit: robot erc_panel, 64 links, 66 joints
Links:
- link indicator_1_led_link: geometry collision mesh filename=file:///home/misara/Simulation_ws/src/ROAR-26-Simulation/in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 scale=0.001 0.001 0.001; visual mesh filename=file:///home/misara/Simulation_ws/src/ROAR-26-Simulation/in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 scale=0.001 0.001 0.001
- link indicator_1_link: geometry collision mesh filename=file:///home/misara/Simulation_ws/src/ROAR-26-Simulation/in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 scale=0.001 0.001 0.001; visual mesh filename=file:///home/misara/Simulation_ws/src/ROAR-26-Simulation/in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 scale=0.001 0.001 0.001
- link indicator_2_led_link: geometry collision mesh filename=file:///home/misara/Simulation_ws/src/ROAR-26-Simulation/in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 scale=0.001 0.001 0.001; visual mesh filename=file:///home/misara/Simulation_ws/src/ROAR-26-Simulation/in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 scale=0.001 0.001 0.001
- link indicator_2_link: geometry collision mesh filename=file:///home/misara/Simulation_ws/src/ROAR-26-Simulation/in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 scale=0.001 0.001 0.001; visual mesh filename=file:///home/misara/Simulation_ws/src/ROAR-26-Simulation/in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 scale=0.001 0.001 0.001
- link indicator_3_led_link: geometry collision mesh filename=file:///home/misara/Simulation_ws/src/ROAR-26-Simulation/in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 scale=0.001 0.001 0.001; visual mesh filename=file:///home/misara/Simulation_ws/src/ROAR-26-Simulation/in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 scale=0.001 0.001 0.001
- link indicator_3_link: geometry collision mesh filename=file:///home/misara/Simulation_ws/src/ROAR-26-Simulation/in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 scale=0.001 0.001 0.001; visual mesh filename=file:///home/misara/Simulation_ws/src/ROAR-26-Simulation/in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 scale=0.001 0.001 0.001
- link indicator_4_led_link: geometry collision mesh filename=file:///home/misara/Simulation_ws/src/ROAR-26-Simulation/in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 scale=0.001 0.001 0.001; visual mesh filename=file:///home/misara/Simulation_ws/src/ROAR-26-Simulation/in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 scale=0.001 0.001 0.001
- link indicator_4_link: geometry collision mesh filename=file:///home/misara/Simulation_ws/src/ROAR-26-Simulation/in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 scale=0.001 0.001 0.001; visual mesh filename=file:///home/misara/Simulation_ws/src/ROAR-26-Simulation/in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 scale=0.001 0.001 0.001
- link indicator_5_led_link: geometry collision mesh filename=file:///home/misara/Simulation_ws/src/ROAR-26-Simulation/in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 scale=0.001 0.001 0.001; visual mesh filename=file:///home/misara/Simulation_ws/src/ROAR-26-Simulation/in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 scale=0.001 0.001 0.001
- link indicator_5_link: geometry collision mesh filename=file:///home/misara/Simulation_ws/src/ROAR-26-Simulation/in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 scale=0.001 0.001 0.001; visual mesh filename=file:///home/misara/Simulation_ws/src/ROAR-26-Simulation/in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 scale=0.001 0.001 0.001
- link large_rotary_1_base_link: geometry collision mesh filename=file:///home/misara/Simulation_ws/src/ROAR-26-Simulation/in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 scale=0.001 0.001 0.001; visual mesh filename=file:///home/misara/Simulation_ws/src/ROAR-26-Simulation/in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 scale=0.001 0.001 0.001
- link large_rotary_1_link: geometry collision mesh filename=file:///home/misara/Simulation_ws/src/ROAR-26-Simulation/in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 scale=0.001 0.001 0.001; visual mesh filename=file:///home/misara/Simulation_ws/src/ROAR-26-Simulation/in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 scale=0.001 0.001 0.001
- link large_rotary_2_base_link: geometry collision mesh filename=file:///home/misara/Simulation_ws/src/ROAR-26-Simulation/in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 scale=0.001 0.001 0.001; visual mesh filename=file:///home/misara/Simulation_ws/src/ROAR-26-Simulation/in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 scale=0.001 0.001 0.001
- link large_rotary_2_link: geometry collision mesh filename=file:///home/misara/Simulation_ws/src/ROAR-26-Simulation/in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 scale=0.001 0.001 0.001; visual mesh filename=file:///home/misara/Simulation_ws/src/ROAR-26-Simulation/in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 scale=0.001 0.001 0.001
- link main_switch_link: geometry collision mesh filename=file:///home/misara/Simulation_ws/src/ROAR-26-Simulation/in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 scale=0.001 0.001 0.001; visual mesh filename=file:///home/misara/Simulation_ws/src/ROAR-26-Simulation/in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 scale=0.001 0.001 0.001
- link main_switch_main_link: geometry collision mesh filename=file:///home/misara/Simulation_ws/src/ROAR-26-Simulation/in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 scale=0.001 0.001 0.001; visual mesh filename=file:///home/misara/Simulation_ws/src/ROAR-26-Simulation/in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 scale=0.001 0.001 0.001
- link panel_base_link: geometry collision mesh filename=file:///home/misara/Simulation_ws/src/ROAR-26-Simulation/in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 scale=.001 .001 .001; visual mesh filename=file:///home/misara/Simulation_ws/src/ROAR-26-Simulation/in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 scale=.001 .001 .001
- link rotary_1_knob_link: geometry collision mesh filename=file:///home/misara/Simulation_ws/src/ROAR-26-Simulation/in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 scale=0.001 0.001 0.001; visual mesh filename=file:///home/misara/Simulation_ws/src/ROAR-26-Simulation/in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 scale=0.001 0.001 0.001
- link rotary_1_link: geometry collision mesh filename=file:///home/misara/Simulation_ws/src/ROAR-26-Simulation/in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 scale=0.001 0.001 0.001; visual mesh filename=file:///home/misara/Simulation_ws/src/ROAR-26-Simulation/in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 scale=0.001 0.001 0.001
- link rotary_2_knob_link: geometry collision mesh filename=file:///home/misara/Simulation_ws/src/ROAR-26-Simulation/in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 scale=0.001 0.001 0.001; visual mesh filename=file:///home/misara/Simulation_ws/src/ROAR-26-Simulation/in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 scale=0.001 0.001 0.001
- link rotary_2_link: geometry collision mesh filename=file:///home/misara/Simulation_ws/src/ROAR-26-Simulation/in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 scale=0.001 0.001 0.001; visual mesh filename=file:///home/misara/Simulation_ws/src/ROAR-26-Simulation/in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 scale=0.001 0.001 0.001
- link rotary_3_knob_link: geometry collision mesh filename=file:///home/misara/Simulation_ws/src/ROAR-26-Simulation/in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 scale=0.001 0.001 0.001; visual mesh filename=file:///home/misara/Simulation_ws/src/ROAR-26-Simulation/in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 scale=0.001 0.001 0.001
- link rotary_3_link: geometry collision mesh filename=file:///home/misara/Simulation_ws/src/ROAR-26-Simulation/in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 scale=0.001 0.001 0.001; visual mesh filename=file:///home/misara/Simulation_ws/src/ROAR-26-Simulation/in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 scale=0.001 0.001 0.001
- link rotary_4_knob_link: geometry collision mesh filename=file:///home/misara/Simulation_ws/src/ROAR-26-Simulation/in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 scale=0.001 0.001 0.001; visual mesh filename=file:///home/misara/Simulation_ws/src/ROAR-26-Simulation/in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 scale=0.001 0.001 0.001
- link rotary_4_link: geometry collision mesh filename=file:///home/misara/Simulation_ws/src/ROAR-26-Simulation/in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 scale=0.001 0.001 0.001; visual mesh filename=file:///home/misara/Simulation_ws/src/ROAR-26-Simulation/in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 scale=0.001 0.001 0.001
- link rotary_5_knob_link: geometry collision mesh filename=file:///home/misara/Simulation_ws/src/ROAR-26-Simulation/in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 scale=0.001 0.001 0.001; visual mesh filename=file:///home/misara/Simulation_ws/src/ROAR-26-Simulation/in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 scale=0.001 0.001 0.001
- link rotary_5_link: geometry collision mesh filename=file:///home/misara/Simulation_ws/src/ROAR-26-Simulation/in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 scale=0.001 0.001 0.001; visual mesh filename=file:///home/misara/Simulation_ws/src/ROAR-26-Simulation/in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 scale=0.001 0.001 0.001
- link row_10_link: geometry collision mesh filename=file:///home/misara/Simulation_ws/src/ROAR-26-Simulation/in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 scale=0.001 0.001 0.001; visual mesh filename=file:///home/misara/Simulation_ws/src/ROAR-26-Simulation/in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 scale=0.001 0.001 0.001
- link row_10_row_link: geometry collision mesh filename=file:///home/misara/Simulation_ws/src/ROAR-26-Simulation/in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 scale=0.001 0.001 0.001; visual mesh filename=file:///home/misara/Simulation_ws/src/ROAR-26-Simulation/in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 scale=0.001 0.001 0.001
- link row_11_link: geometry collision mesh filename=file:///home/misara/Simulation_ws/src/ROAR-26-Simulation/in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 scale=0.001 0.001 0.001; visual mesh filename=file:///home/misara/Simulation_ws/src/ROAR-26-Simulation/in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 scale=0.001 0.001 0.001
- link row_11_row_link: geometry collision mesh filename=file:///home/misara/Simulation_ws/src/ROAR-26-Simulation/in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 scale=0.001 0.001 0.001; visual mesh filename=file:///home/misara/Simulation_ws/src/ROAR-26-Simulation/in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 scale=0.001 0.001 0.001
- link row_12_link: geometry collision mesh filename=file:///home/misara/Simulation_ws/src/ROAR-26-Simulation/in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 scale=0.001 0.001 0.001; visual mesh filename=file:///home/misara/Simulation_ws/src/ROAR-26-Simulation/in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 scale=0.001 0.001 0.001
- link row_12_row_link: geometry collision mesh filename=file:///home/misara/Simulation_ws/src/ROAR-26-Simulation/in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 scale=0.001 0.001 0.001; visual mesh filename=file:///home/misara/Simulation_ws/src/ROAR-26-Simulation/in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 scale=0.001 0.001 0.001
- link row_13_link: geometry collision mesh filename=file:///home/misara/Simulation_ws/src/ROAR-26-Simulation/in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 scale=0.001 0.001 0.001; visual mesh filename=file:///home/misara/Simulation_ws/src/ROAR-26-Simulation/in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 scale=0.001 0.001 0.001
- link row_13_row_link: geometry collision mesh filename=file:///home/misara/Simulation_ws/src/ROAR-26-Simulation/in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 scale=0.001 0.001 0.001; visual mesh filename=file:///home/misara/Simulation_ws/src/ROAR-26-Simulation/in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 scale=0.001 0.001 0.001
- link row_1_link: geometry collision mesh filename=file:///home/misara/Simulation_ws/src/ROAR-26-Simulation/in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 scale=0.001 0.001 0.001; visual mesh filename=file:///home/misara/Simulation_ws/src/ROAR-26-Simulation/in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 scale=0.001 0.001 0.001
- link row_1_row_link: geometry collision mesh filename=file:///home/misara/Simulation_ws/src/ROAR-26-Simulation/in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 scale=0.001 0.001 0.001; visual mesh filename=file:///home/misara/Simulation_ws/src/ROAR-26-Simulation/in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 scale=0.001 0.001 0.001
- link row_2_link: geometry collision mesh filename=file:///home/misara/Simulation_ws/src/ROAR-26-Simulation/in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 scale=0.001 0.001 0.001; visual mesh filename=file:///home/misara/Simulation_ws/src/ROAR-26-Simulation/in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 scale=0.001 0.001 0.001
- link row_2_row_link: geometry collision mesh filename=file:///home/misara/Simulation_ws/src/ROAR-26-Simulation/in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 scale=0.001 0.001 0.001; visual mesh filename=file:///home/misara/Simulation_ws/src/ROAR-26-Simulation/in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 scale=0.001 0.001 0.001
- link row_3_link: geometry collision mesh filename=file:///home/misara/Simulation_ws/src/ROAR-26-Simulation/in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 scale=0.001 0.001 0.001; visual mesh filename=file:///home/misara/Simulation_ws/src/ROAR-26-Simulation/in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 scale=0.001 0.001 0.001
- link row_3_row_link: geometry collision mesh filename=file:///home/misara/Simulation_ws/src/ROAR-26-Simulation/in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 scale=0.001 0.001 0.001; visual mesh filename=file:///home/misara/Simulation_ws/src/ROAR-26-Simulation/in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 scale=0.001 0.001 0.001
- link row_4_link: geometry collision mesh filename=file:///home/misara/Simulation_ws/src/ROAR-26-Simulation/in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 scale=0.001 0.001 0.001; visual mesh filename=file:///home/misara/Simulation_ws/src/ROAR-26-Simulation/in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 scale=0.001 0.001 0.001
- link row_4_row_link: geometry collision mesh filename=file:///home/misara/Simulation_ws/src/ROAR-26-Simulation/in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 scale=0.001 0.001 0.001; visual mesh filename=file:///home/misara/Simulation_ws/src/ROAR-26-Simulation/in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 scale=0.001 0.001 0.001
- link row_5_link: geometry collision mesh filename=file:///home/misara/Simulation_ws/src/ROAR-26-Simulation/in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 scale=0.001 0.001 0.001; visual mesh filename=file:///home/misara/Simulation_ws/src/ROAR-26-Simulation/in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 scale=0.001 0.001 0.001
- link row_5_row_link: geometry collision mesh filename=file:///home/misara/Simulation_ws/src/ROAR-26-Simulation/in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 scale=0.001 0.001 0.001; visual mesh filename=file:///home/misara/Simulation_ws/src/ROAR-26-Simulation/in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 scale=0.001 0.001 0.001
- link row_6_link: geometry collision mesh filename=file:///home/misara/Simulation_ws/src/ROAR-26-Simulation/in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 scale=0.001 0.001 0.001; visual mesh filename=file:///home/misara/Simulation_ws/src/ROAR-26-Simulation/in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 scale=0.001 0.001 0.001
- link row_6_row_link: geometry collision mesh filename=file:///home/misara/Simulation_ws/src/ROAR-26-Simulation/in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 scale=0.001 0.001 0.001; visual mesh filename=file:///home/misara/Simulation_ws/src/ROAR-26-Simulation/in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 scale=0.001 0.001 0.001
- link row_7_link: geometry collision mesh filename=file:///home/misara/Simulation_ws/src/ROAR-26-Simulation/in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 scale=0.001 0.001 0.001; visual mesh filename=file:///home/misara/Simulation_ws/src/ROAR-26-Simulation/in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 scale=0.001 0.001 0.001
- link row_7_row_link: geometry collision mesh filename=file:///home/misara/Simulation_ws/src/ROAR-26-Simulation/in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 scale=0.001 0.001 0.001; visual mesh filename=file:///home/misara/Simulation_ws/src/ROAR-26-Simulation/in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 scale=0.001 0.001 0.001
- link row_8_link: geometry collision mesh filename=file:///home/misara/Simulation_ws/src/ROAR-26-Simulation/in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 scale=0.001 0.001 0.001; visual mesh filename=file:///home/misara/Simulation_ws/src/ROAR-26-Simulation/in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 scale=0.001 0.001 0.001
- link row_8_row_link: geometry collision mesh filename=file:///home/misara/Simulation_ws/src/ROAR-26-Simulation/in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 scale=0.001 0.001 0.001; visual mesh filename=file:///home/misara/Simulation_ws/src/ROAR-26-Simulation/in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 scale=0.001 0.001 0.001
- link row_9_link: geometry collision mesh filename=file:///home/misara/Simulation_ws/src/ROAR-26-Simulation/in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 scale=0.001 0.001 0.001; visual mesh filename=file:///home/misara/Simulation_ws/src/ROAR-26-Simulation/in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 scale=0.001 0.001 0.001
- link row_9_row_link: geometry collision mesh filename=file:///home/misara/Simulation_ws/src/ROAR-26-Simulation/in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 scale=0.001 0.001 0.001; visual mesh filename=file:///home/misara/Simulation_ws/src/ROAR-26-Simulation/in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 scale=0.001 0.001 0.001
- link slab_link: geometry collision mesh filename=file:///home/misara/Simulation_ws/src/ROAR-26-Simulation/in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 scale=0.001 0.001 0.001; visual mesh filename=file:///home/misara/Simulation_ws/src/ROAR-26-Simulation/in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 scale=0.001 0.001 0.001
- link socket_1_link: geometry collision mesh filename=file:///home/misara/Simulation_ws/src/ROAR-26-Simulation/in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 scale=0.001 0.001 0.001; visual mesh filename=file:///home/misara/Simulation_ws/src/ROAR-26-Simulation/in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 scale=0.001 0.001 0.001
- link socket_2_link: geometry collision mesh filename=file:///home/misara/Simulation_ws/src/ROAR-26-Simulation/in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 scale=0.001 0.001 0.001; visual mesh filename=file:///home/misara/Simulation_ws/src/ROAR-26-Simulation/in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 scale=0.001 0.001 0.001

File: panel/src/electromagnet_description/urdf/electromagnet.xacro (robot description, xacro)
@@ -2,7 +2,7 @@
 <robot name="electromagnet" xmlns:xacro="http://www.ros.org/wiki/xacro">
 <!--<xacro:include filename="$(find electromagnet_description)/urdf/materials.xacro" />-->
-<xacro:include filename="$(find electromagnet_description)/urdf/electromagnet.ros2control" />
 <xacro:include filename="$(find electromagnet_description)/urdf/electromagnet.gazebo" />
 <xacro:macro name="electromagnet" params="name parent x y z">
+<xacro:include filename="$(find electromagnet_description)/urdf/electromagnet.ros2control" />
 <link name="${name}_link">
   <inertial>

File: panel/src/led_indicator_description/urdf/led_indicator.xacro (robot description, xacro)
@@ -2,7 +2,7 @@
 <robot name="led_indicator" xmlns:xacro="http://www.ros.org/wiki/xacro">
 <!-- <xacro:include filename="$(find led_indicator_description)/urdf/materials.xacro" /> -->
-<xacro:include filename="$(find led_indicator_description)/urdf/led_indicator.ros2control" />
 <xacro:include filename="$(find led_indicator_description)/urdf/led_indicator.gazebo" />
 <xacro:macro name="led_indicator" params="name parent x y z">
+<xacro:include filename="$(find led_indicator_description)/urdf/led_indicator.ros2control" />
 <link name="${name}_link">
   <inertial>

File: panel/src/main_switch_description/urdf/main_switch.xacro (robot description, xacro)
@@ -2,7 +2,7 @@
 <robot name="main_switch" xmlns:xacro="http://www.ros.org/wiki/xacro">
 <!-- <xacro:include filename="$(find main_switch_description)/urdf/materials.xacro" /> -->
-<xacro:include filename="$(find main_switch_description)/urdf/main_switch.ros2control" />
 <xacro:include filename="$(find main_switch_description)/urdf/main_switch.gazebo" />
 <xacro:macro name="main_switch" params="name parent x y z">
+<xacro:include filename="$(find main_switch_description)/urdf/main_switch.ros2control" />
 <link name="${name}_link">
   <inertial>

File: panel/src/rotary_description/urdf/rotary.xacro (robot description, xacro)
@@ -2,7 +2,7 @@
 <robot name="rotary" xmlns:xacro="http://www.ros.org/wiki/xacro">
 <!-- <xacro:include filename="$(find rotary_description)/urdf/rotary_materials.xacro" />  color defined in main xacro now-->
-<xacro:include filename="$(find rotary_description)/urdf/rotary.ros2control" />
 <xacro:include filename="$(find rotary_description)/urdf/rotary.gazebo" />
 <xacro:macro name="rotary" params="name parent x y z">
+<xacro:include filename="$(find rotary_description)/urdf/rotary.ros2control" />
 <link name="${name}_base_link">
   <inertial>

File: panel/src/row_description/urdf/row.xacro (robot description, xacro)
@@ -2,7 +2,7 @@
 <robot name="row" xmlns:xacro="http://www.ros.org/wiki/xacro">
 <!-- xacro:include filename="$(find row_description)/urdf/materials.xacro" /> -->
-<xacro:include filename="$(find row_description)/urdf/row.ros2control" />
 <xacro:include filename="$(find row_description)/urdf/row.gazebo" />
 <xacro:macro name="row" params="name parent x y z">
+<xacro:include filename="$(find row_description)/urdf/row.ros2control" />
 <link name="${name}_link">
   <inertial>

File: panel/src/slab_description/urdf/slab.xacro (robot description, xacro)
@@ -2,7 +2,7 @@
 <robot name="slab" xmlns:xacro="http://www.ros.org/wiki/xacro">
 <!--<xacro:include filename="$(find slab_description)/urdf/materials.xacro" />-->
-<xacro:include filename="$(find slab_description)/urdf/slab.ros2control" />
 <xacro:include filename="$(find slab_description)/urdf/slab.gazebo" />
 <xacro:macro name="slab" params="name parent x y z">
+<xacro:include filename="$(find slab_description)/urdf/slab.ros2control" />
 <link name="${name}_link">
   <inertial>

File: panel/src/socket_description/urdf/socket.xacro (robot description, xacro)
@@ -2,7 +2,7 @@
 <robot name="socket" xmlns:xacro="http://www.ros.org/wiki/xacro">
 <!-- <xacro:include filename="$(find socket_description)/urdf/materials.xacro" /> -->
-<xacro:include filename="$(find socket_description)/urdf/socket.ros2control" />
 <xacro:include filename="$(find socket_description)/urdf/socket.gazebo" />
 <xacro:macro name="socket" params="name parent x y z">
+<xacro:include filename="$(find socket_description)/urdf/socket.ros2control" />
 <link name="${name}_link">
   <inertial>

File: panel/src/switch_description/urdf/rotary_control.xacro (robot description, xacro)
@@ -2,8 +2,8 @@
 <robot name="switch" xmlns:xacro="http://www.ros.org/wiki/xacro">
 <!-- <xacro:include filename="$(find switch_description)/urdf/switch_materials.xacro" />  color defined in main xacro now-->
-<xacro:include filename="$(find switch_description)/urdf/switch.ros2control" />
 <xacro:include filename="$(find switch_description)/urdf/switch.gazebo" />
 <!-- added the next line to define {name} and be able to call it multiple times in the main urdf file -->
 <xacro:macro name="rotary_switch" params="name parent x y z">
+  <xacro:include filename="$(find switch_description)/urdf/switch.ros2control" />
   <link name="${name}_link">
     <inertial>
