Commit message: Adjust panel body collision geometry and physics optimizations

File: panel/src/electromagnet_description/urdf/electromagnet.xacro (robot description, xacro)
@@ -19,7 +19,8 @@
   </visual>
   <collision>
-    <origin xyz="0 0 0" rpy="0 0 0"/>
+    <!-- Box approximation of electromagnet bracket (24.5×140×30 mm), centred at mesh centroid -->
+    <origin xyz="0.0 0.0 0.01500" rpy="0 0 0"/>
     <geometry>
-      <mesh filename="file://$(find electromagnet_description)/meshes/magnet_base_link.stl" scale="0.001 0.001 0.001"/>
+      <box size="0.02452 0.14000 0.03000"/>
     </geometry>
   </collision>
@@ -39,7 +40,9 @@
   </visual>
   <collision>
-    <origin xyz="-0.0 -0.0 -0.03" rpy="0 0 0"/>
+    <!-- Box approximation of magnet disc (51.8×230×20 mm) -->
+    <!-- visual offset (0,0,-0.03) + mesh centroid (0,0,0.02) = (0,0,-0.01) -->
+    <origin xyz="0.0 0.0 -0.01" rpy="0 0 0"/>
     <geometry>
-      <mesh filename="file://$(find electromagnet_description)/meshes/magnet_link.stl" scale="0.001 0.001 0.001"/>
+      <box size="0.05177 0.23000 0.02000"/>
     </geometry>
   </collision>

File: panel/src/erc_panel_sim/worlds/led_indicator.xacro (robot description, xacro)
@@ -19,7 +19,8 @@
   </visual>
   <collision>
-    <origin xyz="0 0 0" rpy="0 0 0"/>
+    <!-- Box approximation of LED body housing (27.2×16.2×11.55 mm), centred at mesh centroid -->
+    <origin xyz="0.0 0.0 0.01607" rpy="0 0 0"/>
     <geometry>
-      <mesh filename="file://$(find led_indicator_description)/meshes/led_base_link.stl" scale="0.001 0.001 0.001"/>
+      <box size="0.0272 0.0162 0.0115"/>
     </geometry>
   </collision>
@@ -39,7 +40,9 @@
   </visual>
   <collision>
-    <origin xyz="-0.0 0.0 -0.007566" rpy="0 0 0"/>
+    <!-- Box approximation of LED lens cap (27.2×12.8×9.65 mm) -->
+    <!-- visual offset (0,0,-0.007566) + mesh centroid (0,0,0.01623) = (0,0,0.008664) -->
+    <origin xyz="0.0 0.0 0.008664" rpy="0 0 0"/>
     <geometry>
-      <mesh filename="file://$(find led_indicator_description)/meshes/led_link.stl" scale="0.001 0.001 0.001"/>
+      <box size="0.0272 0.0128 0.0096"/>
     </geometry>
   </collision>

File: panel/src/led_indicator_description/urdf/led_indicator.xacro (robot description, xacro)
@@ -19,7 +19,9 @@
   </visual>
   <collision>
-    <origin xyz="0 0 0" rpy="0 0 0"/>
+    <!-- Box approximation of LED body housing (27.2×16.2×11.55 mm), centred at mesh centroid -->
+    <!-- mesh centroid at z=0.01607 m above origin -->
+    <origin xyz="0.0 0.0 0.01607" rpy="0 0 0"/>
     <geometry>
-      <mesh filename="file://$(find led_indicator_description)/meshes/led_base_link.stl" scale="0.001 0.001 0.001"/>
+      <box size="0.0272 0.0162 0.0115"/>
     </geometry>
   </collision>
@@ -39,7 +41,9 @@
   </visual>
   <collision>
-    <origin xyz="-0.0 0.0 -0.007566" rpy="0 0 0"/>
+    <!-- Box approximation of LED lens cap (27.2×12.8×9.65 mm) -->
+    <!-- visual offset (0,0,-0.007566) + mesh centroid (0,0,0.01623) = (0,0,0.008664) -->
+    <origin xyz="0.0 0.0 0.008664" rpy="0 0 0"/>
     <geometry>
-      <mesh filename="file://$(find led_indicator_description)/meshes/led_link.stl" scale="0.001 0.001 0.001"/>
+      <box size="0.0272 0.0128 0.0096"/>
     </geometry>
   </collision>

File: panel/src/main_switch_description/urdf/main_switch.xacro (robot description, xacro)
@@ -19,7 +19,8 @@
   </visual>
   <collision>
-    <origin xyz="0 0 0" rpy="0 0 0"/>
+    <!-- Box approximation of main switch body (71.5×74×91 mm), centred at mesh centroid -->
+    <origin xyz="-0.00326 0.01492 0.00349" rpy="0 0 0"/>
     <geometry>
-      <mesh filename="file://$(find main_switch_description)/meshes/main_base_link.stl" scale="0.001 0.001 0.001"/>
+      <box size="0.0715 0.0740 0.0911"/>
     </geometry>
   </collision>
@@ -39,7 +40,10 @@
   </visual>
   <collision>
-    <origin xyz="0.023986 0.010731 -0.00361" rpy="0 0 0"/>
+    <!-- Box approximation of main switch lever (16.5×19.4×17.3 mm) -->
+    <!-- visual offset (0.023986, 0.010731, -0.00361) + mesh centroid (0.02399, -0.01875, -0.00093) -->
+    <!-- combined: (0.02399+0.023986, 0.010731-0.01875, -0.00361-0.00093) = (0.04797, -0.00802, -0.00454) -->
+    <origin xyz="0.04797 -0.00802 -0.00454" rpy="0 0 0"/>
     <geometry>
-      <mesh filename="file://$(find main_switch_description)/meshes/main_link.stl" scale="0.001 0.001 0.001"/>
+      <box size="0.0165 0.0194 0.0173"/>
     </geometry>
   </collision>

File: panel/src/rotary_description/urdf/rotary.xacro (robot description, xacro)
@@ -19,7 +19,8 @@
   </visual>
   <collision>
-    <origin xyz="0 0 0" rpy="0 0 0"/>
+    <!-- Box approximation of large rotary base (68.6×86.3×72.1 mm), centred at mesh centroid -->
+    <origin xyz="0.00021 0.02536 0.03570" rpy="0 0 0"/>
     <geometry>
-      <mesh filename="file://$(find rotary_description)/meshes/rotary_base_link.stl" scale="0.001 0.001 0.001"/>
+      <box size="0.0686 0.0863 0.0721"/>
     </geometry>
   </collision>
@@ -39,7 +40,10 @@
   </visual>
   <collision>
-    <origin xyz="-0.000209 -0.052756 -0.033931" rpy="0 0 0"/>
+    <!-- Cylinder approximation of rotary knob (r≈21 mm, h≈28.5 mm), axis along Y -->
+    <!-- visual origin is (-0.000209, -0.052756, -0.033931); mesh centroid at cy=0.06698 m -->
+    <!-- combined: visual_origin + mesh_centroid_offset = (-0.000209, 0.01422, -0.00031) -->
+    <origin xyz="-0.000209 0.01422 -0.00031" rpy="1.5708 0 0"/>
     <geometry>
-      <mesh filename="file://$(find rotary_description)/meshes/rotary_link.stl" scale="0.001 0.001 0.001"/>
+      <cylinder radius="0.021" length="0.0285"/>
     </geometry>
   </collision>

File: panel/src/row_description/urdf/row.xacro (robot description, xacro)
@@ -19,7 +19,8 @@
   </visual>
   <collision>
-    <origin xyz="0 0 0" rpy="0 0 0"/>
+    <!-- Box approximation of toggle-switch base (20.4×68.8×85.6 mm), centred at mesh centroid -->
+    <origin xyz="0.00006 -0.01561 -0.00182" rpy="0 0 0"/>
     <geometry>
-      <mesh filename="file://$(find row_description)/meshes/row_base_link.stl" scale="0.001 0.001 0.001"/>
+      <box size="0.0204 0.0688 0.0856"/>
     </geometry>
   </collision>
@@ -39,7 +40,10 @@
   </visual>
   <collision>
-    <origin xyz="-5.6e-05 -0.017761 0.008932" rpy="0 0 0"/>
+    <!-- Box approximation of toggle lever (17.1×6.9×14.7 mm) -->
+    <!-- visual offset (-5.6e-05, -0.017761, 0.008932) + mesh centroid (0.00006, 0.01847, -0.01087) -->
+    <!-- combined Y: -0.017761 + 0.01847 = 0.000709  Z: 0.008932 - 0.01087 = -0.001938 -->
+    <origin xyz="0.0 0.000709 -0.001938" rpy="0 0 0"/>
     <geometry>
-      <mesh filename="file://$(find row_description)/meshes/row_link.stl" scale="0.001 0.001 0.001"/>
+      <box size="0.0171 0.0069 0.0147"/>
     </geometry>
   </collision>

File: panel/src/slab_description/urdf/slab.xacro (robot description, xacro)
@@ -19,7 +19,8 @@
   </visual>
   <collision>
-    <origin xyz="0 0 0" rpy="0 0 0"/>
+    <!-- Box approximation of slab holder (40.25×200×105 mm), centred at mesh centroid -->
+    <origin xyz="0.00095 -0.00062 0.05056" rpy="0 0 0"/>
     <geometry>
-      <mesh filename="file://$(find slab_description)/meshes/slab_base_link.stl" scale="0.001 0.001 0.001"/>
+      <box size="0.04025 0.20000 0.10500"/>
     </geometry>
   </collision>

File: panel/src/socket_description/urdf/socket.xacro (robot description, xacro)
@@ -19,7 +19,8 @@
   </visual>
   <collision>
-    <origin xyz="0 0 0" rpy="0 0 0"/>
+    <!-- Box approximation of IEC socket body (49×22×26.5 mm), centred at mesh centroid -->
+    <origin xyz="0.00017 0.00032 -0.00663" rpy="0 0 0"/>
     <geometry>
-      <mesh filename="file://$(find socket_description)/meshes/socket_base_link.stl" scale="0.001 0.001 0.001"/>
+      <box size="0.0490 0.0220 0.0265"/>
     </geometry>
   </collision>

File: panel/src/switch_description/urdf/rotary_control.xacro (robot description, xacro)
@@ -20,7 +20,8 @@
     </visual>
     <collision>
-      <origin xyz="0 0 0" rpy="0 0 0"/>
+      <!-- Box approximation of switch body (30x52.5x43.8 mm), centered at mesh centroid -->
+      <origin xyz="0.0 -0.01525 0.00109" rpy="0 0 0"/>
       <geometry>
-        <mesh filename="file://$(find switch_description)/meshes/base_link.stl" scale="0.001 0.001 0.001"/> <!-- changed the mesh to base_link.stl ashan el mesh sabet -->
+        <box size="0.030 0.0525 0.0438"/>
       </geometry>
     </collision>
@@ -40,7 +41,9 @@
     </visual>
     <collision>
-      <origin xyz="-0.0 -0.008 -0.0" rpy="0 0 0"/>
+      <!-- Cylinder approximation of rotary knob (r=12mm, l=26mm), axis along X -->
+      <!-- visual offset is -0.008 in Y; knob mesh center is at Y=+0.01525 → combined Y = 0.00725 -->
+      <origin xyz="0.0 0.00725 -0.001" rpy="0 1.5708 0"/>
       <geometry>
-        <mesh filename="file://$(find switch_description)/meshes/knob_link_1_1.stl" scale="0.001 0.001 0.001"/> <!-- changed the mesh to knob_link_1_1.stl ashan el mesh sabet -->
+        <cylinder radius="0.012" length="0.026"/>
       </geometry>
     </collision>
