Commit message: mostafamostafamostafa

File: dev_environment/rover/roar_rover_clean/urdf/modules/rover_gazebo.xacro (robot description, xacro)
@@ -6,4 +6,13 @@
         <parameters>${controllers_yaml}</parameters>
       </plugin>
+    </gazebo>
+    <gazebo reference="base_link">
+      <sensor name="chassis_contact" type="contact">
+        <contact>
+          <collision>base_footprint_fixed_joint_lump__base_link_collision</collision>
+        </contact>
+        <update_rate>10</update_rate>
+        <topic>/chassis/contact_sensors</topic>
+      </sensor>
     </gazebo>
   </xacro:macro>

File: dev_environment/rover/roar_rover_noise/urdf/modules/rover_gazebo.xacro (robot description, xacro)
@@ -6,4 +6,13 @@
         <parameters>${controllers_yaml}</parameters>
       </plugin>
+    </gazebo>
+    <gazebo reference="base_link">
+      <sensor name="chassis_contact" type="contact">
+        <contact>
+          <collision>base_footprint_fixed_joint_lump__base_link_collision</collision>
+        </contact>
+        <update_rate>10</update_rate>
+        <topic>/chassis/contact_sensors</topic>
+      </sensor>
     </gazebo>
   </xacro:macro>
