Commit message: Add collision alarm node and contact sensors for all rover configs, and removed build files

File: dev_environment/rover/roar_rover_clean/backups/ros1/rover_gazebo.xacro (robot description, xacro)
@@ -89,4 +89,5 @@
         <plugin name="camera_plugin" filename="libgazebo_ros_depth_camera.so">
           <always_on>true</always_on>
+        <topic>/rover_contact</topic>
           <update_rate>0.0</update_rate>
           <frameName>camera_depth_optical_frame</frameName>
@@ -127,4 +128,23 @@
       </plugin>
     </gazebo>
+    <xacro:contact_sensor_gazebo name="base_link" />
+    <xacro:contact_sensor_gazebo name="wheel_rhs_front" />
+    <xacro:contact_sensor_gazebo name="wheel_rhs_mid" />
+    <xacro:contact_sensor_gazebo name="wheel_rhs_rear" />
+    <xacro:contact_sensor_gazebo name="wheel_lhs_front" />
+    <xacro:contact_sensor_gazebo name="wheel_lhs_mid" />
+    <xacro:contact_sensor_gazebo name="wheel_lhs_rear" />
+  </xacro:macro>
+  <xacro:macro name="contact_sensor_gazebo" params="name">
+    <gazebo reference="${name}">
+      <sensor name="${name}_contact" type="contact">
+        <always_on>true</always_on>
+        <topic>/rover_contact</topic>
+        <update_rate>50</update_rate>
+        <contact>
+          <collision>${name}_collision</collision>
+        </contact>
+      </sensor>
+    </gazebo>
   </xacro:macro>
 </robot>

File: dev_environment/rover/roar_rover_clean/urdf/modules/rover_gazebo.xacro (robot description, xacro)
@@ -7,11 +7,21 @@
       </plugin>
     </gazebo>
-    <gazebo reference="base_link">
-      <sensor name="chassis_contact" type="contact">
+    <xacro:contact_sensor_gazebo name="base_link" />
+    <xacro:contact_sensor_gazebo name="wheel_rhs_front" />
+    <xacro:contact_sensor_gazebo name="wheel_rhs_mid" />
+    <xacro:contact_sensor_gazebo name="wheel_rhs_rear" />
+    <xacro:contact_sensor_gazebo name="wheel_lhs_front" />
+    <xacro:contact_sensor_gazebo name="wheel_lhs_mid" />
+    <xacro:contact_sensor_gazebo name="wheel_lhs_rear" />
+  </xacro:macro>
+  <xacro:macro name="contact_sensor_gazebo" params="name">
+    <gazebo reference="${name}">
+      <sensor name="${name}_contact" type="contact">
+        <always_on>true</always_on>
+        <topic>/rover_contact</topic>
+        <update_rate>50</update_rate>
         <contact>
-          <collision>base_footprint_fixed_joint_lump__base_link_collision</collision>
+          <collision>${name}_collision</collision>
         </contact>
-        <update_rate>10</update_rate>
-        <topic>/chassis/contact_sensors</topic>
       </sensor>
     </gazebo>

File: dev_environment/rover/roar_rover_clean/urdf/modules/rover_gazebo_clean.xacro (robot description, xacro)
@@ -6,4 +6,23 @@
         <parameters>${controllers_yaml}</parameters>
       </plugin>
+    </gazebo>
+    <xacro:contact_sensor_gazebo name="base_link" />
+    <xacro:contact_sensor_gazebo name="wheel_rhs_front" />
+    <xacro:contact_sensor_gazebo name="wheel_rhs_mid" />
+    <xacro:contact_sensor_gazebo name="wheel_rhs_rear" />
+    <xacro:contact_sensor_gazebo name="wheel_lhs_front" />
+    <xacro:contact_sensor_gazebo name="wheel_lhs_mid" />
+    <xacro:contact_sensor_gazebo name="wheel_lhs_rear" />
+  </xacro:macro>
+  <xacro:macro name="contact_sensor_gazebo" params="name">
+    <gazebo reference="${name}">
+      <sensor name="${name}_contact" type="contact">
+        <always_on>true</always_on>
+        <topic>/rover_contact</topic>
+        <update_rate>50</update_rate>
+        <contact>
+          <collision>${name}_collision</collision>
+        </contact>
+      </sensor>
     </gazebo>
   </xacro:macro>

File: dev_environment/rover/roar_rover_noise/urdf/modules/rover_gazebo.xacro (robot description, xacro)
@@ -7,11 +7,21 @@
       </plugin>
     </gazebo>
-    <gazebo reference="base_link">
-      <sensor name="chassis_contact" type="contact">
+    <xacro:contact_sensor_gazebo name="base_link" />
+    <xacro:contact_sensor_gazebo name="wheel_rhs_front" />
+    <xacro:contact_sensor_gazebo name="wheel_rhs_mid" />
+    <xacro:contact_sensor_gazebo name="wheel_rhs_rear" />
+    <xacro:contact_sensor_gazebo name="wheel_lhs_front" />
+    <xacro:contact_sensor_gazebo name="wheel_lhs_mid" />
+    <xacro:contact_sensor_gazebo name="wheel_lhs_rear" />
+  </xacro:macro>
+  <xacro:macro name="contact_sensor_gazebo" params="name">
+    <gazebo reference="${name}">
+      <sensor name="${name}_contact" type="contact">
+        <always_on>true</always_on>
+        <topic>/rover_contact</topic>
+        <update_rate>50</update_rate>
         <contact>
-          <collision>base_footprint_fixed_joint_lump__base_link_collision</collision>
+          <collision>${name}_collision</collision>
         </contact>
-        <update_rate>10</update_rate>
-        <topic>/chassis/contact_sensors</topic>
       </sensor>
     </gazebo>

File: rover/roar_rover_clean/urdf/modules/rover_gazebo.xacro (robot description, xacro)
@@ -6,4 +6,23 @@
         <parameters>${controllers_yaml}</parameters>
       </plugin>
+    </gazebo>
+    <xacro:contact_sensor_gazebo name="base_link" />
+    <xacro:contact_sensor_gazebo name="wheel_rhs_front" />
+    <xacro:contact_sensor_gazebo name="wheel_rhs_mid" />
+    <xacro:contact_sensor_gazebo name="wheel_rhs_rear" />
+    <xacro:contact_sensor_gazebo name="wheel_lhs_front" />
+    <xacro:contact_sensor_gazebo name="wheel_lhs_mid" />
+    <xacro:contact_sensor_gazebo name="wheel_lhs_rear" />
+  </xacro:macro>
+  <xacro:macro name="contact_sensor_gazebo" params="name">
+    <gazebo reference="${name}">
+      <sensor name="${name}_contact" type="contact">
+        <always_on>true</always_on>
+        <topic>/rover_contact</topic>
+        <update_rate>50</update_rate>
+        <contact>
+          <collision>${name}_collision</collision>
+        </contact>
+      </sensor>
     </gazebo>
   </xacro:macro>
